Commit message: feat: 3-robot zigzag conveyor system with parallel belts
- Implemented 3 parallel conveyor belts (Belt 1, 2, 3) with unique namespaces
- Added fleet_manager package for scalable multi-robot coordination
- Configured zigzag robot layout: R1 (west) -> Belt1 -> R2 (center) -> Belt2 -> R3 (west) -> Belt3
- Robot positions: R1 and R3 aligned at y=-0.5, R2 at y=0.8
- Created start_conveyors.sh script for async belt control
- Belt 2 flows in reverse direction for zigzag pattern
- Added break beam sensors at belt ends
- Integrated robot_interface with state machine and handoff coordination
- Added pick area and accumulation tables

Fixes: Robot positioning, conveyor plugin namespace conflicts, sensor placement

File: src/xarm_ros2/xarm_description/urdf/common/common.gazebo.xacro (robot description, xacro)
@@ -11,8 +11,13 @@
     </gazebo>
   </xacro:macro>
-  <xacro:macro name="gazebo_ros2_control_plugin" params="ros2_control_params:=''">
+  <xacro:macro name="gazebo_ros2_control_plugin" params="ros2_control_params:='' ros_namespace:=''">
     <gazebo>
       <plugin filename="libgazebo_ros2_control.so" name="gazebo_ros2_control">
         <robot_sim_type>gazebo_ros2_control/GazeboSystem</robot_sim_type>
+        <xacro:if value="${ros_namespace != ''}">
+          <ros>
+            <namespace>${ros_namespace}</namespace>
+          </ros>
+        </xacro:if>
         <xacro:if value="${ros2_control_params != ''}">
           <parameters>${ros2_control_params}</parameters>

File: src/xarm_ros2/xarm_description/urdf/xarm_device.urdf.xacro (robot description, xacro)
@@ -39,4 +39,5 @@
   <xacro:arg name="mesh_suffix" default="stl"/>
   <xacro:arg name="kinematics_suffix" default=""/>
+  <xacro:arg name="ros_namespace" default=""/>
   <!-- load xarm device -->
   <xacro:include filename="$(find xarm_description)/urdf/xarm_device_macro.xacro" />
@@ -59,4 +60,4 @@
     baud_checkset="$(arg baud_checkset)" default_gripper_baud="$(arg default_gripper_baud)"
     model1300="$(arg model1300)" attach_to="$(arg attach_to)" attach_xyz="$(arg attach_xyz)" attach_rpy="$(arg attach_rpy)"
-    robot_sn="$(arg robot_sn)" use_gazebo_camera="$(arg use_gazebo_camera)" mesh_suffix="$(arg mesh_suffix)" kinematics_suffix="$(arg kinematics_suffix)" />
+    robot_sn="$(arg robot_sn)" use_gazebo_camera="$(arg use_gazebo_camera)" mesh_suffix="$(arg mesh_suffix)" kinematics_suffix="$(arg kinematics_suffix)" ros_namespace="$(arg ros_namespace)" />
 </robot>

File: src/xarm_ros2/xarm_description/urdf/xarm_device_macro.xacro (robot description, xacro)
@@ -42,4 +42,5 @@
     mesh_suffix:='stl'
     kinematics_suffix:=''
+    ros_namespace:=''
     "
     >
@@ -283,5 +284,5 @@
         </xacro:if>
         <xacro:if value="${ros2_control_plugin == 'gazebo_ros2_control/GazeboSystem'}">
-          <xacro:gazebo_ros2_control_plugin ros2_control_params="${new_ros2_control_params}"/>
+          <xacro:gazebo_ros2_control_plugin ros2_control_params="${new_ros2_control_params}" ros_namespace="${ros_namespace}"/>
         </xacro:if>
       </xacro:if>
