Commit message: fix(L0/L1): make the model's geometry and its frames describe one cell
Phase 1.C. Closes C1, H1, H2, H3, M-07, M-08, M-09, M-11, M-12, M-13, R-17,
R-06/H9 and R-14 from the review fan-out on feature/phase-1.

The critical defect: belt_1200x400 declared a 0.100 m collision box while its
surface, infeed and outfeed frames were all at z = 0.600, so the belt's declared
work surface floated half a metre above its geometry. station_transfer_1 places
onto conveyor_1/infeed, so PlaceAt released the work-piece into empty air, and
the break beam could never be broken. The belt is now a 0.600 m body with an
exact recomputed centroidal tensor, and validate/geometric gained
`frame-outside-geometry`, which rejects any named frame outside its own type's
collision box.

The same coordinate was also live twice and 0.3 m apart. generate/description
emitted type frames at `xyz - half_height`, which would only be right if the
link origin were the box centre; the anchor joint puts it at the foot. One
convention now, plus a test asserting every L0 frame resolves to the same world
pose as a URDF link and as a static transform. generate/frames now reads
NamedFrame.link and skips frames a robot description already publishes, so
cell_a__arm_N__tcp is no longer a static transform sitting 0.836 m from the
tool centre point.

Nothing was anchored to the world: `gz sdf -p` produced a 315.75 kg free body
for the cell and three free arm roots. The scene is now static and each arm
carries a fixed joint to `world`, emitted inside <gazebo> so robot_state_
publisher never sees it and no frame gains a second parent. Verified with
sdformat on the real generated descriptions.

Also: mass is declared at the centroid rather than at the foot (lumped cell CoM
moves from z = 0.002 to z = 0.301); a planning-scene collision-object artifact
is generated from the same resolved bodies as the scene, though no runtime node
reads it yet; the sensor housings move out of the gripper's approach corridor
and down to a height a work-piece can interrupt; the tables are given real
clearance; the acceleration ceiling and controller-manager rate move from
generator constants into the robot type (P5); and the determinism check now
regenerates in a fresh interpreter under a different PYTHONHASHSEED, which is
the only place its stated failure mode can occur.

Two scenario defects that were geometry-dependent: pick_and_place asserted a net
rise across a cycle whose pick and place frames are at the same height, so it
could only pass when the cycle failed partway; it now samples height during the
cycle and asserts arrival at the resolved place frame. bringup's
test_no_joint_name_is_shared_between_arms built its own strings and could not
fail; it now reads the live joint_states of all three arms.

No seed reaches any generated artifact, because none can. `gz sim` takes a seed
as a command-line flag rather than an SDF element, and MoveIt exposes no way to
seed OMPL's RNG at all. bringup's dead `cls.seed` is removed; pick_and_place
keeps its read, which feeds the failure report, and both files now state that
the exported seed is consumed by nothing rather than claiming determinism. The
move_group teardown exemption's claim to be a characterised upstream segfault is
replaced with the contradictory evidence actually observed (-11 in one set of
runs, -15 in another); the exemption itself is left unchanged, as that defect is
owned elsewhere.

File: workspace/src/cite_generated/description/cell_a_arm_1.urdf.xacro (robot description, xacro)
@@ -52,4 +52,24 @@
     </plugin>
   </gazebo>
+  <!-- Bolt the arm to the world.
+       `create_attach_link` is false and `arm_1_mount` is not the name
+       the URDF-to-SDF converter anchors on, so without this the arm's root is a
+       free rigid body standing on its pedestal by contact friction alone. Joint
+       reaction torques slide or tip it, and the symptom — base drift — reads as
+       a calibration fault.
+       The joint lives inside a `gazebo` block rather than as a URDF joint to a
+       link named `world`, and that placement is the whole point: a URDF `world`
+       link would make `robot_state_publisher` publish `world` -> mount as a
+       second parent for a frame the generated static transform table already
+       parents to `cite_world`. One frame, two parents, intermittently wrong.
+       Inside `gazebo` the converter sees it and TF never does.
+       The joint carries no pose. Where the arm stands is stated once, by the
+       spawn pose in the bring-up plan; a pose here would apply it twice. -->
+  <gazebo>
+    <joint name="arm_1_mount_world_anchor" type="fixed">
+      <parent>world</parent>
+      <child>arm_1_mount</child>
+    </joint>
+  </gazebo>
   <gazebo>
     <plugin filename="gz_ros2_control-system" name="gz_ros2_control::GazeboSimROS2ControlPlugin">

File: workspace/src/cite_generated/description/cell_a_arm_2.urdf.xacro (robot description, xacro)
@@ -52,4 +52,24 @@
     </plugin>
   </gazebo>
+  <!-- Bolt the arm to the world.
+       `create_attach_link` is false and `arm_2_mount` is not the name
+       the URDF-to-SDF converter anchors on, so without this the arm's root is a
+       free rigid body standing on its pedestal by contact friction alone. Joint
+       reaction torques slide or tip it, and the symptom — base drift — reads as
+       a calibration fault.
+       The joint lives inside a `gazebo` block rather than as a URDF joint to a
+       link named `world`, and that placement is the whole point: a URDF `world`
+       link would make `robot_state_publisher` publish `world` -> mount as a
+       second parent for a frame the generated static transform table already
+       parents to `cite_world`. One frame, two parents, intermittently wrong.
+       Inside `gazebo` the converter sees it and TF never does.
+       The joint carries no pose. Where the arm stands is stated once, by the
+       spawn pose in the bring-up plan; a pose here would apply it twice. -->
+  <gazebo>
+    <joint name="arm_2_mount_world_anchor" type="fixed">
+      <parent>world</parent>
+      <child>arm_2_mount</child>
+    </joint>
+  </gazebo>
   <gazebo>
     <plugin filename="gz_ros2_control-system" name="gz_ros2_control::GazeboSimROS2ControlPlugin">

File: workspace/src/cite_generated/description/cell_a_arm_3.urdf.xacro (robot description, xacro)
@@ -52,4 +52,24 @@
     </plugin>
   </gazebo>
+  <!-- Bolt the arm to the world.
+       `create_attach_link` is false and `arm_3_mount` is not the name
+       the URDF-to-SDF converter anchors on, so without this the arm's root is a
+       free rigid body standing on its pedestal by contact friction alone. Joint
+       reaction torques slide or tip it, and the symptom — base drift — reads as
+       a calibration fault.
+       The joint lives inside a `gazebo` block rather than as a URDF joint to a
+       link named `world`, and that placement is the whole point: a URDF `world`
+       link would make `robot_state_publisher` publish `world` -> mount as a
+       second parent for a frame the generated static transform table already
+       parents to `cite_world`. One frame, two parents, intermittently wrong.
+       Inside `gazebo` the converter sees it and TF never does.
+       The joint carries no pose. Where the arm stands is stated once, by the
+       spawn pose in the bring-up plan; a pose here would apply it twice. -->
+  <gazebo>
+    <joint name="arm_3_mount_world_anchor" type="fixed">
+      <parent>world</parent>
+      <child>arm_3_mount</child>
+    </joint>
+  </gazebo>
   <gazebo>
     <plugin filename="gz_ros2_control-system" name="gz_ros2_control::GazeboSimROS2ControlPlugin">

File: workspace/src/cite_generated/description/cell_a_scene.urdf.xacro (robot description, xacro)
@@ -6,4 +6,19 @@
      ./scripts/validate-model, which diffs this tree against a fresh generator run. -->
 <robot xmlns:xacro="http://ros.org/wiki/xacro" name="cell_a">
+  <!-- Anchor the cell furniture to the world.
+       Every link below is joined by a fixed joint, so converting this URDF to
+       SDF lumps the whole cell into ONE link. Without this the simulator gets a
+       single free rigid body of a few hundred kilograms resting on the ground
+       plane by contact friction alone: joint reaction torques from three arms
+       slide it, and the symptom is base drift that reads as a calibration fault
+       and gets debugged in the wrong layer.
+       `static` rather than a fixed joint to a link named `world`: nothing here
+       has a joint that moves, and a `world` link would also become a second TF
+       parent for every body — `robot_state_publisher` would publish it
+       alongside the generated static transform table, giving one frame two
+       parents. Static costs the physics engine nothing and changes no name. -->
+  <gazebo>
+    <static>true</static>
+  </gazebo>
   <!-- The facility root. Tied to the surveyed physical origin (L5); every frame
        below is expressed relative to it. -->
@@ -12,5 +27,9 @@
   <link name="beam_c1_out_base_link">
     <inertial>
-      <origin xyz="0 0 0" rpy="0 0 0"/>
+      <!-- The body's pose names the point it stands on, so the mass sits half a
+           height above the link origin. `com_m` is measured from the box centre
+           and the tensor beside it is centroidal; declaring both at the foot
+           states a centroidal tensor about a point up to 0.3 m from the mass. -->
+      <origin xyz="0 0 0.06" rpy="0 0 0"/>
       <mass value="0.25"/>
       <inertia ixx="0.00033333" ixy="0"
@@ -30,5 +49,5 @@
     <parent link="cite_world"/>
     <child link="beam_c1_out_base_link"/>
-    <origin xyz="1.6 0 0.68" rpy="0 0 0"/>
+    <origin xyz="1.6 0.25 0.63" rpy="0 0 0"/>
   </joint>
   <link name="beam_c1_out_beam"/>
@@ -36,10 +55,14 @@
     <parent link="beam_c1_out_base_link"/>
     <child link="beam_c1_out_beam"/>
-    <origin xyz="0 0 -0.06" rpy="0 0 0"/>
+    <origin xyz="0 0 0" rpy="0 0 0"/>
   </joint>
   <!-- beam_c2_out — break_beam -->
   <link name="beam_c2_out_base_link">
     <inertial>
-      <origin xyz="0 0 0" rpy="0 0 0"/>
+      <!-- The body's pose names the point it stands on, so the mass sits half a
+           height above the link origin. `com_m` is measured from the box centre
+           and the tensor beside it is centroidal; declaring both at the foot
+           states a centroidal tensor about a point up to 0.3 m from the mass. -->
+      <origin xyz="0 0 0.06" rpy="0 0 0"/>
       <mass value="0.25"/>
       <inertia ixx="0.00033333" ixy="0"
@@ -59,5 +82,5 @@
     <parent link="cite_world"/>
     <child link="beam_c2_out_base_link"/>
-    <origin xyz="3.7 0 0.68" rpy="0 0 0"/>
+    <origin xyz="3.7 0.25 0.63" rpy="0 0 0"/>
   </joint>
   <link name="beam_c2_out_beam"/>
@@ -65,10 +88,14 @@
     <parent link="beam_c2_out_base_link"/>
     <child link="beam_c2_out_beam"/>
-    <origin xyz="0 0 -0.06" rpy="0 0 0"/>
+    <origin xyz="0 0 0" rpy="0 0 0"/>
   </joint>
   <!-- beam_c3_out — break_beam -->
   <link name="beam_c3_out_base_link">
     <inertial>
-      <origin xyz="0 0 0" rpy="0 0 0"/>
+      <!-- The body's pose names the point it stands on, so the mass sits half a
+           height above the link origin. `com_m` is measured from the box centre
+           and the tensor beside it is centroidal; declaring both at the foot
+           states a centroidal tensor about a point up to 0.3 m from the mass. -->
+      <origin xyz="0 0 0.06" rpy="0 0 0"/>
       <mass value="0.25"/>
       <inertia ixx="0.00033333" ixy="0"
@@ -88,5 +115,5 @@
     <parent link="cite_world"/>
     <child link="beam_c3_out_base_link"/>
-    <origin xyz="5.8 0 0.68" rpy="0 0 0"/>
+    <origin xyz="5.8 0.25 0.63" rpy="0 0 0"/>
   </joint>
   <link name="beam_c3_out_beam"/>
@@ -94,22 +121,26 @@
     <parent link="beam_c3_out_base_link"/>
     <child link="beam_c3_out_beam"/>
-    <origin xyz="0 0 -0.06" rpy="0 0 0"/>
+    <origin xyz="0 0 0" rpy="0 0 0"/>
   </joint>
   <!-- conveyor_1 — belt_1200x400 -->
   <link name="conveyor_1_base_link">
     <inertial>
-      <origin xyz="0 0 0" rpy="0 0 0"/>
+      <!-- The body's pose names the point it stands on, so the mass sits half a
+           height above the link origin. `com_m` is measured from the box centre
+           and the tensor beside it is centroidal; declaring both at the foot
+           states a centroidal tensor about a point up to 0.3 m from the mass. -->
+      <origin xyz="0 0 0.3" rpy="0 0 0"/>
       <mass value="45"/>
-      <inertia ixx="0.6375" ixy="0"
-               ixz="0" iyy="5.4375"
+      <inertia ixx="1.95" ixy="0"
+               ixz="0" iyy="6.75"
                iyz="0" izz="6"/>
     </inertial>
     <visual>
-      <origin xyz="0 0 0.05" rpy="0 0 0"/>
-      <geometry><box size="1.2 0.4 0.1"/></geometry>
-    </visual>
-    <collision>
-      <origin xyz="0 0 0.05" rpy="0 0 0"/>
-      <geometry><box size="1.2 0.4 0.1"/></geometry>
+      <origin xyz="0 0 0.3" rpy="0 0 0"/>
+      <geometry><box size="1.2 0.4 0.6"/></geometry>
+    </visual>
+    <collision>
+      <origin xyz="0 0 0.3" rpy="0 0 0"/>
+      <geometry><box size="1.2 0.4 0.6"/></geometry>
     </collision>
   </link>
@@ -123,5 +154,5 @@
     <parent link="conveyor_1_base_link"/>
     <child link="conveyor_1_infeed"/>
-    <origin xyz="-0.6 0 0.55" rpy="0 0 0"/>
+    <origin xyz="-0.6 0 0.6" rpy="0 0 0"/>
   </joint>
   <link name="conveyor_1_outfeed"/>
@@ -129,5 +160,5 @@
     <parent link="conveyor_1_base_link"/>
     <child link="conveyor_1_outfeed"/>
-    <origin xyz="0.6 0 0.55" rpy="0 0 0"/>
+    <origin xyz="0.6 0 0.6" rpy="0 0 0"/>
   </joint>
   <link name="conveyor_1_surface"/>
@@ -135,22 +166,26 @@
     <parent link="conveyor_1_base_link"/>
     <child link="conveyor_1_surface"/>
-    <origin xyz="0 0 0.55" rpy="0 0 0"/>
+    <origin xyz="0 0 0.6" rpy="0 0 0"/>
   </joint>
   <!-- conveyor_2 — belt_1200x400 -->
   <link name="conveyor_2_base_link">
     <inertial>
-      <origin xyz="0 0 0" rpy="0 0 0"/>
+      <!-- The body's pose names the point it stands on, so the mass sits half a
+           height above the link origin. `com_m` is measured from the box centre
+           and the tensor beside it is centroidal; declaring both at the foot
+           states a centroidal tensor about a point up to 0.3 m from the mass. -->
+      <origin xyz="0 0 0.3" rpy="0 0 0"/>
       <mass value="45"/>
-      <inertia ixx="0.6375" ixy="0"
-               ixz="0" iyy="5.4375"
+      <inertia ixx="1.95" ixy="0"
+               ixz="0" iyy="6.75"
                iyz="0" izz="6"/>
     </inertial>
     <visual>
-      <origin xyz="0 0 0.05" rpy="0 0 0"/>
-      <geometry><box size="1.2 0.4 0.1"/></geometry>
-    </visual>
-    <collision>
-      <origin xyz="0 0 0.05" rpy="0 0 0"/>
-      <geometry><box size="1.2 0.4 0.1"/></geometry>
+      <origin xyz="0 0 0.3" rpy="0 0 0"/>
+      <geometry><box size="1.2 0.4 0.6"/></geometry>
+    </visual>
+    <collision>
+      <origin xyz="0 0 0.3" rpy="0 0 0"/>
+      <geometry><box size="1.2 0.4 0.6"/></geometry>
     </collision>
   </link>
@@ -164,5 +199,5 @@
     <parent link="conveyor_2_base_link"/>
     <child link="conveyor_2_infeed"/>
-    <origin xyz="-0.6 0 0.55" rpy="0 0 0"/>
+    <origin xyz="-0.6 0 0.6" rpy="0 0 0"/>
   </joint>
   <link name="conveyor_2_outfeed"/>
@@ -170,5 +205,5 @@
     <parent link="conveyor_2_base_link"/>
     <child link="conveyor_2_outfeed"/>
-    <origin xyz="0.6 0 0.55" rpy="0 0 0"/>
+    <origin xyz="0.6 0 0.6" rpy="0 0 0"/>
   </joint>
   <link name="conveyor_2_surface"/>
@@ -176,22 +211,26 @@
     <parent link="conveyor_2_base_link"/>
     <child link="conveyor_2_surface"/>
-    <origin xyz="0 0 0.55" rpy="0 0 0"/>
+    <origin xyz="0 0 0.6" rpy="0 0 0"/>
   </joint>
   <!-- conveyor_3 — belt_1200x400 -->
   <link name="conveyor_3_base_link">
     <inertial>
-      <origin xyz="0 0 0" rpy="0 0 0"/>
+      <!-- The body's pose names the point it stands on, so the mass sits half a
+           height above the link origin. `com_m` is measured from the box centre
+           and the tensor beside it is centroidal; declaring both at the foot
+           states a centroidal tensor about a point up to 0.3 m from the mass. -->
+      <origin xyz="0 0 0.3" rpy="0 0 0"/>
       <mass value="45"/>
-      <inertia ixx="0.6375" ixy="0"
-               ixz="0" iyy="5.4375"
+      <inertia ixx="1.95" ixy="0"
+               ixz="0" iyy="6.75"
                iyz="0" izz="6"/>
     </inertial>
     <visual>
-      <origin xyz="0 0 0.05" rpy="0 0 0"/>
-      <geometry><box size="1.2 0.4 0.1"/></geometry>
-    </visual>
-    <collision>
-      <origin xyz="0 0 0.05" rpy="0 0 0"/>
-      <geometry><box size="1.2 0.4 0.1"/></geometry>
+      <origin xyz="0 0 0.3" rpy="0 0 0"/>
+      <geometry><box size="1.2 0.4 0.6"/></geometry>
+    </visual>
+    <collision>
+      <origin xyz="0 0 0.3" rpy="0 0 0"/>
+      <geometry><box size="1.2 0.4 0.6"/></geometry>
     </collision>
   </link>
@@ -205,5 +244,5 @@
     <parent link="conveyor_3_base_link"/>
     <child link="conveyor_3_infeed"/>
-    <origin xyz="-0.6 0 0.55" rpy="0 0 0"/>
+    <origin xyz="-0.6 0 0.6" rpy="0 0 0"/>
   </joint>
   <link name="conveyor_3_outfeed"/>
@@ -211,5 +250,5 @@
     <parent link="conveyor_3_base_link"/>
     <child link="conveyor_3_outfeed"/>
-    <origin xyz="0.6 0 0.55" rpy="0 0 0"/>
+    <origin xyz="0.6 0 0.6" rpy="0 0 0"/>
   </joint>
   <link name="conveyor_3_surface"/>
@@ -217,10 +256,14 @@
     <parent link="conveyor_3_base_link"/>
     <child link="conveyor_3_surface"/>
-    <origin xyz="0 0 0.55" rpy="0 0 0"/>
+    <origin xyz="0 0 0.6" rpy="0 0 0"/>
   </joint>
   <!-- pedestal_1 — pedestal_600 -->
   <link name="pedestal_1_base_link">
     <inertial>
-      <origin xyz="0 0 0" rpy="0 0 0"/>
+      <!-- The body's pose names the point it stands on, so the mass sits half a
+           height above the link origin. `com_m` is measured from the box centre
+           and the tensor beside it is centroidal; declaring both at the foot
+           states a centroidal tensor about a point up to 0.3 m from the mass. -->
+      <origin xyz="0 0 0.3" rpy="0 0 0"/>
       <mass value="40"/>
       <inertia ixx="1.5" ixy="0"
@@ -246,10 +289,14 @@
     <parent link="pedestal_1_base_link"/>
     <child link="pedestal_1_top"/>
-    <origin xyz="0 0 0.3" rpy="0 0 0"/>
+    <origin xyz="0 0 0.6" rpy="0 0 0"/>
   </joint>
   <!-- pedestal_2 — pedestal_600 -->
   <link name="pedestal_2_base_link">
     <inertial>
-      <origin xyz="0 0 0" rpy="0 0 0"/>
+      <!-- The body's pose names the point it stands on, so the mass sits half a
+           height above the link origin. `com_m` is measured from the box centre
+           and the tensor beside it is centroidal; declaring both at the foot
+           states a centroidal tensor about a point up to 0.3 m from the mass. -->
+      <origin xyz="0 0 0.3" rpy="0 0 0"/>
       <mass value="40"/>
       <inertia ixx="1.5" ixy="0"
@@ -275,10 +322,14 @@
     <parent link="pedestal_2_base_link"/>
     <child link="pedestal_2_top"/>
-    <origin xyz="0 0 0.3" rpy="0 0 0"/>
+    <origin xyz="0 0 0.6" rpy="0 0 0"/>
   </joint>
   <!-- pedestal_3 — pedestal_600 -->
   <link name="pedestal_3_base_link">
     <inertial>
-      <origin xyz="0 0 0" rpy="0 0 0"/>
+      <!-- The body's pose names the point it stands on, so the mass sits half a
+           height above the link origin. `com_m` is measured from the box centre
+           and the tensor beside it is centroidal; declaring both at the foot
+           states a centroidal tensor about a point up to 0.3 m from the mass. -->
+      <origin xyz="0 0 0.3" rpy="0 0 0"/>
       <mass value="40"/>
       <inertia ixx="1.5" ixy="0"
@@ -304,10 +355,14 @@
     <parent link="pedestal_3_base_link"/>
     <child link="pedestal_3_top"/>
-    <origin xyz="0 0 0.3" rpy="0 0 0"/>
+    <origin xyz="0 0 0.6" rpy="0 0 0"/>
   </joint>
   <!-- table_accumulation — work_table_600 -->
   <link name="table_accumulation_base_link">
     <inertial>
-      <origin xyz="0 0 0" rpy="0 0 0"/>
+      <!-- The body's pose names the point it stands on, so the mass sits half a
+           height above the link origin. `com_m` is measured from the box centre
+           and the tensor beside it is centroidal; declaring both at the foot
+           states a centroidal tensor about a point up to 0.3 m from the mass. -->
+      <origin xyz="0 0 0.3" rpy="0 0 0"/>
       <mass value="30"/>
       <inertia ixx="1.8" ixy="0"
@@ -327,5 +382,5 @@
     <parent link="cite_world"/>
     <child link="table_accumulation_base_link"/>
-    <origin xyz="6.15 0 0" rpy="0 0 0"/>
+    <origin xyz="6.2 0 0" rpy="0 0 0"/>
   </joint>
   <link name="table_accumulation_surface"/>
@@ -333,10 +388,14 @@
     <parent link="table_accumulation_base_link"/>
     <child link="table_accumulation_surface"/>
-    <origin xyz="0 0 0.3" rpy="0 0 0"/>
+    <origin xyz="0 0 0.6" rpy="0 0 0"/>
   </joint>
   <!-- table_pick — work_table_600 -->
   <link name="table_pick_base_link">
     <inertial>
-      <origin xyz="0 0 0" rpy="0 0 0"/>
+      <!-- The body's pose names the point it stands on, so the mass sits half a
+           height above the link origin. `com_m` is measured from the box centre
+           and the tensor beside it is centroidal; declaring both at the foot
+           states a centroidal tensor about a point up to 0.3 m from the mass. -->
+      <origin xyz="0 0 0.3" rpy="0 0 0"/>
       <mass value="30"/>
       <inertia ixx="1.8" ixy="0"
@@ -356,5 +415,5 @@
     <parent link="cite_world"/>
     <child link="table_pick_base_link"/>
-    <origin xyz="-0.45 0 0" rpy="0 0 0"/>
+    <origin xyz="-0.475 0 0" rpy="0 0 0"/>
   </joint>
   <link name="table_pick_surface"/>
@@ -362,5 +421,5 @@
     <parent link="table_pick_base_link"/>
     <child link="table_pick_surface"/>
-    <origin xyz="0 0 0.3" rpy="0 0 0"/>
+    <origin xyz="0 0 0.6" rpy="0 0 0"/>
   </joint>
 </robot>
