Commit message: fix(L0): give belt transfer points a real support margin, and a rule that sees it
`./scripts/scenario pick_and_place` failed 0 of 18 deterministically because
`cell_a__conveyor_1__infeed` lay exactly on the belt's leading-edge plane. A
50 mm cube released there has its centre of mass projecting onto the boundary of
its support polygon — neutrally stable — so it tipped about the edge and fell
0.6 m to the floor, while the release itself succeeded and every layer above
reported so. Six frames shared the fault: all three belts use one type, and both
ends of it.

THE LAYOUT. The transfer frames move 0.050 m inboard of the belt's ends, and the
arm standoff moves from 0.350 m to 0.300 m to pay for the reach it costs. 0.025 m
— exactly half a cube — was rejected: it is the neutral case, not a margin. The
result is 50 mm of support at every transfer point, 25 mm past the tipping
boundary and about 13x the 1.9 mm the release pose was measured accurate to, with
every station at 83.3% of the arm's envelope against an 85% comfort threshold —
better than the 84.3% the pick from table_pick had before. Sliding the belts
instead was rejected: both ends of a belt serve different arms, so it helps one
station and hurts the other. The layout is PROVISIONAL per charter §8, so
re-spacing it now is a model edit rather than a revision of a survey.

THE VALIDATOR COULD NOT SEE THE CLASS, which is the second defect and the reason
the first survived. `_frames_lie_on_their_own_geometry` asks whether a frame is
OUTSIDE its body, with strict comparisons, so a frame on a boundary face passes —
right for a work surface, useless for a work point. It has no notion of support
margin, and could not acquire one: L0 recorded no work-piece geometry.

So L0 gains a work-piece type — `AssetType` category `workpiece`, no instances,
`Facility.workpiece_models` now resolving to it — and two rules are built on it:

  * `insufficient-support-margin` (geometric) requires half the widest
    work-piece plus SUPPORT_CLEARANCE_M of support under every station pick and
    place point. Against the committed frame positions it reports all five
    station points at 0.0 mm against 45.0 mm needed, and does not report
    table_pick's centred surface.
  * `default-grasp-width-never-closes` (physical) re-tightens from 88.93 mm to
    47.86 mm — the narrowest part, less twice the gripper controller's own
    `goal_tolerance` converted through the linkage, which is the same
    discrimination margin `cite_skills::gripper_is_holding` uses. The 88.93 mm
    ceiling was a deliberate loosening from 60.92 mm when ADR-0023's attachment
    plugin was removed, with a note naming the missing part dimensions as the
    blocker; this pays that back.

Comments in model/ and tools/ that asserted the missing-geometry gap are
corrected rather than left standing (P7).

Co-Authored-By: Claude Opus 5 (1M context) <noreply@anthropic.com>
Claude-Session: https://claude.ai/code/session_01DL7n4ktvAptaHzeFAYT1z2

File: workspace/src/cite_generated/description/cell_a_scene.urdf.xacro (robot description, xacro)
@@ -49,5 +49,5 @@
     <parent link="cite_world"/>
     <child link="beam_c1_out_base_link"/>
-    <origin xyz="1.6 0.25 0.63" rpy="0 0 0"/>
+    <origin xyz="1.55 0.25 0.63" rpy="0 0 0"/>
   </joint>
   <link name="beam_c1_out_beam"/>
@@ -82,5 +82,5 @@
     <parent link="cite_world"/>
     <child link="beam_c2_out_base_link"/>
-    <origin xyz="3.7 0.25 0.63" rpy="0 0 0"/>
+    <origin xyz="3.65 0.25 0.63" rpy="0 0 0"/>
   </joint>
   <link name="beam_c2_out_beam"/>
@@ -115,5 +115,5 @@
     <parent link="cite_world"/>
     <child link="beam_c3_out_base_link"/>
-    <origin xyz="5.8 0.25 0.63" rpy="0 0 0"/>
+    <origin xyz="5.75 0.25 0.63" rpy="0 0 0"/>
   </joint>
   <link name="beam_c3_out_beam"/>
@@ -154,5 +154,5 @@
     <parent link="conveyor_1_base_link"/>
     <child link="conveyor_1_infeed"/>
-    <origin xyz="-0.6 0 0.6" rpy="0 0 0"/>
+    <origin xyz="-0.55 0 0.6" rpy="0 0 0"/>
   </joint>
   <link name="conveyor_1_outfeed"/>
@@ -160,5 +160,5 @@
     <parent link="conveyor_1_base_link"/>
     <child link="conveyor_1_outfeed"/>
-    <origin xyz="0.6 0 0.6" rpy="0 0 0"/>
+    <origin xyz="0.55 0 0.6" rpy="0 0 0"/>
   </joint>
   <link name="conveyor_1_surface"/>
@@ -199,5 +199,5 @@
     <parent link="conveyor_2_base_link"/>
     <child link="conveyor_2_infeed"/>
-    <origin xyz="-0.6 0 0.6" rpy="0 0 0"/>
+    <origin xyz="-0.55 0 0.6" rpy="0 0 0"/>
   </joint>
   <link name="conveyor_2_outfeed"/>
@@ -205,5 +205,5 @@
     <parent link="conveyor_2_base_link"/>
     <child link="conveyor_2_outfeed"/>
-    <origin xyz="0.6 0 0.6" rpy="0 0 0"/>
+    <origin xyz="0.55 0 0.6" rpy="0 0 0"/>
   </joint>
   <link name="conveyor_2_surface"/>
@@ -244,5 +244,5 @@
     <parent link="conveyor_3_base_link"/>
     <child link="conveyor_3_infeed"/>
-    <origin xyz="-0.6 0 0.6" rpy="0 0 0"/>
+    <origin xyz="-0.55 0 0.6" rpy="0 0 0"/>
   </joint>
   <link name="conveyor_3_outfeed"/>
@@ -250,5 +250,5 @@
     <parent link="conveyor_3_base_link"/>
     <child link="conveyor_3_outfeed"/>
-    <origin xyz="0.6 0 0.6" rpy="0 0 0"/>
+    <origin xyz="0.55 0 0.6" rpy="0 0 0"/>
   </joint>
   <link name="conveyor_3_surface"/>
@@ -283,5 +283,5 @@
     <parent link="cite_world"/>
     <child link="pedestal_1_base_link"/>
-    <origin xyz="0 -0.35 0" rpy="0 0 0"/>
+    <origin xyz="0 -0.3 0" rpy="0 0 0"/>
   </joint>
   <link name="pedestal_1_top"/>
@@ -316,5 +316,5 @@
     <parent link="cite_world"/>
     <child link="pedestal_2_base_link"/>
-    <origin xyz="2.1 -0.35 0" rpy="0 0 0"/>
+    <origin xyz="2.1 -0.3 0" rpy="0 0 0"/>
   </joint>
   <link name="pedestal_2_top"/>
@@ -349,5 +349,5 @@
     <parent link="cite_world"/>
     <child link="pedestal_3_base_link"/>
-    <origin xyz="4.2 -0.35 0" rpy="0 0 0"/>
+    <origin xyz="4.2 -0.3 0" rpy="0 0 0"/>
   </joint>
   <link name="pedestal_3_top"/>

Commit message: fix(line): give the infeed a sensor, and stop Detect standing in for one
Three findings against the continuous-line scenario, which fails 0 of 4 at
milestone 1 of 9.

R-01, Critical — the line cannot start. `station_transfer_1` was the one
acting station the model gave nothing to observe with. Its cycle fell through
`AwaitTrigger`, whose topic was empty, and came to rest in `DetectAt`, which
`line_tree.hpp` had told to treat an empty result as an idle line and look
again. `Detect` answers an UNOBSERVED region with the same SUCCESS and the same
empty list as an observed empty one — its own detail says "this is not a report
that the region is empty" — and `Detect.action` carries no code separating the
two, so the poll could never end. Measured: WORKING with occupancy 0/1, for as
long as the scenario would wait.

Fixed in L0, because a station that acts must observe: `beam_pick` stands on
the pick table at the same +0.250 m offset every other beam uses, which is the
side away from the arms and outside the 0.100 m corridor the gripper descends
through. The alternative — letting a source-fed station pick without observing
— was rejected: nothing else bounds its cycle, so an empty table would send the
arm down to check and burn the station's retry budget doing it.

The polling path is then removed rather than left unused. `DetectAt` loses the
`require_immediate` port, `line_tree.hpp` emits no attribute for it, and
`line_station.xml` binds none: an empty detection is always a reported failure
with a structured code, and waiting for work is `AwaitTrigger`'s alone.

R-01b, Critical, measured while confirming the above and previously unreported
— NO station could see its own beam. `DetectAt` asked for a 0.30 m region,
which is a half-extent of 0.150 m, against beams the geometric validator forces
to stand 0.250 m off every pick frame. All three acting stations were affected,
not just the infeed; nothing caught it because `cite_skills`'s contract tests
send a 100 m region on purpose and `pick_and_place` never calls `Detect`. The
stand-in is now 0.60 m and `test_detection_region.py` pins both bounds against
the generated frames, reading the number out of the header rather than
restating it.

R-03, Major — the coordinator aborted on its cancellation path.
`SkillNode::abandon` called `async_cancel_goal` on a handle the client had
already forgotten, which throws `UnknownGoalHandleError` on the tick thread
where nothing caught it. The window is ordinary: `rclcpp_action::Client` sets
the handle's result and then erases it, on the executor's thread, so a leaf
halted between its last poll and its next tick cancels a goal that has ended.
Reachable on every halt — recovery and preemption, not only shutdown. A goal
that has already ended is this function's own post-condition arriving early, so
it is now checked for and caught, and reported rather than swallowed.

Two host tooling tests listed the cell's inventory a second time and failed for
saying so; both now derive it from the model.

R-02, the belt timing, is NOT addressed here and needs an ADR. See the fix
report.

Co-Authored-By: Claude Opus 5 (1M context) <noreply@anthropic.com>
Claude-Session: https://claude.ai/code/session_01DL7n4ktvAptaHzeFAYT1z2

File: workspace/src/cite_generated/description/cell_a_scene.urdf.xacro (robot description, xacro)
@@ -123,4 +123,37 @@
     <origin xyz="0 0 0" rpy="0 0 0"/>
   </joint>
+  <!-- beam_pick — break_beam -->
+  <link name="beam_pick_base_link">
+    <inertial>
+      <!-- The body's pose names the point it stands on, so the mass sits half a
+           height above the link origin. `com_m` is measured from the box centre
+           and the tensor beside it is centroidal; declaring both at the foot
+           states a centroidal tensor about a point up to 0.3 m from the mass. -->
+      <origin xyz="0 0 0.06" rpy="0 0 0"/>
+      <mass value="0.25"/>
+      <inertia ixx="0.00033333" ixy="0"
+               ixz="0" iyy="0.00033333"
+               iyz="0" izz="6.667e-05"/>
+    </inertial>
+    <visual>
+      <origin xyz="0 0 0.06" rpy="0 0 0"/>
+      <geometry><box size="0.04 0.04 0.12"/></geometry>
+    </visual>
+    <collision>
+      <origin xyz="0 0 0.06" rpy="0 0 0"/>
+      <geometry><box size="0.04 0.04 0.12"/></geometry>
+    </collision>
+  </link>
+  <joint name="beam_pick_anchor" type="fixed">
+    <parent link="cite_world"/>
+    <child link="beam_pick_base_link"/>
+    <origin xyz="-0.475 0.25 0.63" rpy="0 0 0"/>
+  </joint>
+  <link name="beam_pick_beam"/>
+  <joint name="beam_pick_beam_fixed" type="fixed">
+    <parent link="beam_pick_base_link"/>
+    <child link="beam_pick_beam"/>
+    <origin xyz="0 0 0" rpy="0 0 0"/>
+  </joint>
   <!-- conveyor_1 — belt_1200x400 -->
   <link name="conveyor_1_base_link">

Commit message: fix(L1): the break beam intersects the part's body, not its origin
A through beam breaks on a work-piece's leading edge and stays broken until
its trailing edge is past, at any height the part reaches. The plugin tested
the part's model ORIGIN against a box instead, which was wrong in two
directions and both were measured:

  * across the beam, the origin test gave the sensor a window of part-CENTRE
    heights — a part between 20 mm and 100 mm tall. Anything outside that is
    detected on hardware and was missed here.
  * along the belt, it reported the 50 mm cube 25 mm after its leading edge
    arrived. With the belt indexed on that edge every piece parked 69 mm short
    of arm_2's grasp; the arm closed on air at `commanded 45.0 mm, reached
    46.0 mm, stalled=false` and continuous_line stopped at milestone 4 of 10
    on four runs out of four.

The beam is now a segment tested against the collision shapes the simulator
holds. No work-piece dimension is declared to the plugin or passed into it, so
a part whose size changes in L0 changes what the beam sees (P1, P5).

Getting the physics right does not by itself park the part under the gripper —
a leading-edge break stops it EARLIER, not later. So where an indexing beam is
mounted is now derived rather than authored: half a work-piece plus half a beam
width downstream of the point the part must stop on, which is also how a
photo-eye is set on a physical indexing line. `beam_c1_out` moves from a fitted
-0.050 m to a derived +0.027 m, and a part whose leading edge breaks it comes to
rest with its centre on `conveyor_1/outfeed`.

Sliding the beam until the scenario passed was refused, for the third time. The
old 0.040 m beam width was anti-tunnelling inflation for the origin test, not a
measurement; carrying half of it into L0 geometry would have tuned the layout to
a simulator artefact and left the physical cell parking its parts 20 mm
elsewhere (P2). With the body test the occlusion window is the part's own
length, so the inflation is removed and the width is a real 4 mm aperture.

Four validator rules make this class of defect fail in a second instead of in a
four-run scenario: beam-indexes-off-frame, beam-indexes-no-pick-point,
beam-off-its-belt, beam-cannot-index, plus beam-cannot-see-workpiece for the
height face.

Co-Authored-By: Claude Opus 5 (1M context) <noreply@anthropic.com>
Claude-Session: https://claude.ai/code/session_01DL7n4ktvAptaHzeFAYT1z2

File: workspace/src/cite_generated/description/cell_a_scene.urdf.xacro (robot description, xacro)
@@ -49,5 +49,5 @@
     <parent link="cite_world"/>
     <child link="beam_c1_out_base_link"/>
-    <origin xyz="1.55 0.25 0.63" rpy="0 0 0"/>
+    <origin xyz="1.627 0.25 0.63" rpy="0 0 0"/>
   </joint>
   <link name="beam_c1_out_beam"/>
@@ -82,5 +82,5 @@
     <parent link="cite_world"/>
     <child link="beam_c2_out_base_link"/>
-    <origin xyz="3.65 0.25 0.63" rpy="0 0 0"/>
+    <origin xyz="3.727 0.25 0.63" rpy="0 0 0"/>
   </joint>
   <link name="beam_c2_out_beam"/>
