Commit message: feat(model): a material library in L0, resolved into every visual
The project owner opened the Gazebo GUI and reported that the box, the table
and everything else were black. They were. `Body.material` has carried a name
on every authored body since the component library was written — `table_top`,
`conveyor_frame`, `pedestal_steel`, `sensor_housing`, `workpiece_stock` — and
nothing anywhere resolved it: no library, no rule, no emitter. The generated
scene's every `<visual>` was a bare `<geometry>`, so every renderer fell back to
its own default, and not one line of output said so.

L0 now declares the library, in `model/facility/materials.yaml` beside the other
facility-wide singletons, and the generator resolves it:

* the scene URDF defines each material its bodies wear once at robot scope and
  references it by name in each visual;
* `materials/appearance.yaml` states the library and which body wears what, for
  the one visible object that is in no description — the work-piece, which has
  no instances by design and is spawned into a running world;
* a name no material declares is a referential ERROR, `unknown-material`. A
  warning or a stock-grey default would leave exactly the state above, with the
  cell looking deliberate while the model said something else.

`cite_bringup.workpiece` is now the one statement of the model a work-piece is
spawned as. It was two — a hand-written SDF string in each of the two scenarios
that spawn one, carrying a colour authored nowhere — and it is in a product
package rather than under `tests/` because a scenario is not its only caller.

MODEL_HASH moved, which is correct: the library is model content that reaches a
generated artifact, so a recording stamped with that hash can say what the cell
it was taken from looked like.

NO PHYSICS CHANGED. The work-piece's mass, inertia, friction and geometry are
the literals both scenarios carried, moved unchanged; `test_the_physics_is_
unchanged` is that constraint written where a later edit meets it. URDF carries
one colour where SDF carries two, and sdformat was measured here scaling it by
1.25 and clamping at 1.0 — recorded on the template and the library rather than
compensated for.

Co-Authored-By: Claude Opus 5 (1M context) <noreply@anthropic.com>
Claude-Session: https://claude.ai/code/session_01Vy1FhCAqmLftuxT9L8G4sE

File: workspace/src/cite_generated/description/cell_a_scene.urdf.xacro (robot description, xacro)
@@ -24,4 +24,41 @@
        below is expressed relative to it. -->
   <link name="cite_world"/>
+  <!-- The appearances the bodies below wear, defined once each and referenced by
+       name. Every value is resolved from the facility's material library in L0;
+       nothing here is authored.
+       WHY THESE EXIST AT ALL. Until 2026-09-28 every visual in this file was a
+       bare <geometry> and the cell rendered black, while L0 had carried a
+       material name on each of those bodies the whole time and nothing resolved
+       it.
+       DEFINED HERE AND REFERENCED BELOW, rather than repeated inside each
+       <visual>. urdfdom resolves a name-only <material> against the robot-scope
+       map, so this is the form in which one colour is written once per document
+       — and repeating a definition makes urdfdom warn that the material is not
+       unique and keep whichever it saw first.
+       ONE COLOUR, WHERE L0 DECLARES TWO, AND THE DIFFUSE IS THE ONE THAT SURVIVES.
+       URDF has a single <color> per material and no ambient term. Measured in
+       this project's container on 2026-09-28 with `gz sdf -p` over a probe URDF:
+       sdformat copies this rgba onto BOTH the SDF ambient and the SDF diffuse,
+       after multiplying the three colour components by 1.25 and clamping each at
+       1.0, with alpha untouched. So the declared ambient reaches nothing on this
+       path and the declared diffuse is shown 25% brighter.
+       That is recorded and NOT compensated for. Dividing by 1.25 here would put
+       an undeclared constant in this template that tracks an upstream
+       implementation detail, and what it would buy is cosmetic — nothing in this
+       repository measures a colour. What the library does instead is keep every
+       component a scene body wears at or under 0.8, where the multiply cannot
+       clip; the reason is stated on the library itself. -->
+  <material name="conveyor_frame">
+    <color rgba="0.28 0.34 0.42 1"/>
+  </material>
+  <material name="pedestal_steel">
+    <color rgba="0.52 0.53 0.56 1"/>
+  </material>
+  <material name="sensor_housing">
+    <color rgba="0.78 0.62 0.1 1"/>
+  </material>
+  <material name="table_top">
+    <color rgba="0.58 0.38 0.2 1"/>
+  </material>
   <!-- beam_c1_out — break_beam -->
   <link name="beam_c1_out_base_link">
@@ -40,4 +77,5 @@
       <origin xyz="0 0 0.06" rpy="0 0 0"/>
       <geometry><box size="0.04 0.04 0.12"/></geometry>
+      <material name="sensor_housing"/>
     </visual>
     <collision>
@@ -73,4 +111,5 @@
       <origin xyz="0 0 0.06" rpy="0 0 0"/>
       <geometry><box size="0.04 0.04 0.12"/></geometry>
+      <material name="sensor_housing"/>
     </visual>
     <collision>
@@ -106,4 +145,5 @@
       <origin xyz="0 0 0.06" rpy="0 0 0"/>
       <geometry><box size="0.04 0.04 0.12"/></geometry>
+      <material name="sensor_housing"/>
     </visual>
     <collision>
@@ -139,4 +179,5 @@
       <origin xyz="0 0 0.06" rpy="0 0 0"/>
       <geometry><box size="0.04 0.04 0.12"/></geometry>
+      <material name="sensor_housing"/>
     </visual>
     <collision>
@@ -172,4 +213,5 @@
       <origin xyz="0 0 0.3" rpy="0 0 0"/>
       <geometry><box size="1.2 0.4 0.6"/></geometry>
+      <material name="conveyor_frame"/>
     </visual>
     <collision>
@@ -217,4 +259,5 @@
       <origin xyz="0 0 0.3" rpy="0 0 0"/>
       <geometry><box size="1.2 0.4 0.6"/></geometry>
+      <material name="conveyor_frame"/>
     </visual>
     <collision>
@@ -262,4 +305,5 @@
       <origin xyz="0 0 0.3" rpy="0 0 0"/>
       <geometry><box size="1.2 0.4 0.6"/></geometry>
+      <material name="conveyor_frame"/>
     </visual>
     <collision>
@@ -307,4 +351,5 @@
       <origin xyz="0 0 0.3" rpy="0 0 0"/>
       <geometry><box size="0.3 0.3 0.6"/></geometry>
+      <material name="pedestal_steel"/>
     </visual>
     <collision>
@@ -340,4 +385,5 @@
       <origin xyz="0 0 0.3" rpy="0 0 0"/>
       <geometry><box size="0.3 0.3 0.6"/></geometry>
+      <material name="pedestal_steel"/>
     </visual>
     <collision>
@@ -373,4 +419,5 @@
       <origin xyz="0 0 0.3" rpy="0 0 0"/>
       <geometry><box size="0.3 0.3 0.6"/></geometry>
+      <material name="pedestal_steel"/>
     </visual>
     <collision>
@@ -406,4 +453,5 @@
       <origin xyz="0 0 0.3" rpy="0 0 0"/>
       <geometry><box size="0.6 0.6 0.6"/></geometry>
+      <material name="table_top"/>
     </visual>
     <collision>
@@ -439,4 +487,5 @@
       <origin xyz="0 0 0.3" rpy="0 0 0"/>
       <geometry><box size="0.6 0.6 0.6"/></geometry>
+      <material name="table_top"/>
     </visual>
     <collision>

File: workspace/src/cite_generated/description/cell_b_scene.urdf.xacro (robot description, xacro)
@@ -24,4 +24,41 @@
        below is expressed relative to it. -->
   <link name="cite_world"/>
+  <!-- The appearances the bodies below wear, defined once each and referenced by
+       name. Every value is resolved from the facility's material library in L0;
+       nothing here is authored.
+       WHY THESE EXIST AT ALL. Until 2026-09-28 every visual in this file was a
+       bare <geometry> and the cell rendered black, while L0 had carried a
+       material name on each of those bodies the whole time and nothing resolved
+       it.
+       DEFINED HERE AND REFERENCED BELOW, rather than repeated inside each
+       <visual>. urdfdom resolves a name-only <material> against the robot-scope
+       map, so this is the form in which one colour is written once per document
+       — and repeating a definition makes urdfdom warn that the material is not
+       unique and keep whichever it saw first.
+       ONE COLOUR, WHERE L0 DECLARES TWO, AND THE DIFFUSE IS THE ONE THAT SURVIVES.
+       URDF has a single <color> per material and no ambient term. Measured in
+       this project's container on 2026-09-28 with `gz sdf -p` over a probe URDF:
+       sdformat copies this rgba onto BOTH the SDF ambient and the SDF diffuse,
+       after multiplying the three colour components by 1.25 and clamping each at
+       1.0, with alpha untouched. So the declared ambient reaches nothing on this
+       path and the declared diffuse is shown 25% brighter.
+       That is recorded and NOT compensated for. Dividing by 1.25 here would put
+       an undeclared constant in this template that tracks an upstream
+       implementation detail, and what it would buy is cosmetic — nothing in this
+       repository measures a colour. What the library does instead is keep every
+       component a scene body wears at or under 0.8, where the multiply cannot
+       clip; the reason is stated on the library itself. -->
+  <material name="conveyor_frame">
+    <color rgba="0.28 0.34 0.42 1"/>
+  </material>
+  <material name="pedestal_steel">
+    <color rgba="0.52 0.53 0.56 1"/>
+  </material>
+  <material name="sensor_housing">
+    <color rgba="0.78 0.62 0.1 1"/>
+  </material>
+  <material name="table_top">
+    <color rgba="0.58 0.38 0.2 1"/>
+  </material>
   <!-- infeed_beam — break_beam -->
   <link name="infeed_beam_base_link">
@@ -40,4 +77,5 @@
       <origin xyz="0 0 0.06" rpy="0 0 0"/>
       <geometry><box size="0.04 0.04 0.12"/></geometry>
+      <material name="sensor_housing"/>
     </visual>
     <collision>
@@ -73,4 +111,5 @@
       <origin xyz="0 0 0.3" rpy="0 0 0"/>
       <geometry><box size="0.6 0.6 0.6"/></geometry>
+      <material name="table_top"/>
     </visual>
     <collision>
@@ -106,4 +145,5 @@
       <origin xyz="0 0 0.06" rpy="0 0 0"/>
       <geometry><box size="0.04 0.04 0.12"/></geometry>
+      <material name="sensor_housing"/>
     </visual>
     <collision>
@@ -139,4 +179,5 @@
       <origin xyz="0 0 0.3" rpy="0 0 0"/>
       <geometry><box size="0.6 0.6 0.6"/></geometry>
+      <material name="table_top"/>
     </visual>
     <collision>
@@ -172,4 +213,5 @@
       <origin xyz="0 0 0.3" rpy="0 0 0"/>
       <geometry><box size="0.3 0.3 0.6"/></geometry>
+      <material name="pedestal_steel"/>
     </visual>
     <collision>
@@ -205,4 +247,5 @@
       <origin xyz="0 0 0.3" rpy="0 0 0"/>
       <geometry><box size="1.2 0.4 0.6"/></geometry>
+      <material name="conveyor_frame"/>
     </visual>
     <collision>

Commit message: feat(model): read the real program, put the arm on a linear track, derive the box
L0 now reads the real xArm 5's UFACTORY Studio program instead of poses
taught in simulation (ADR-0067):

- cite_tools.model.blockly reads the Blockly XML strictly: the block types
  the program uses and nothing else; blended moves, moves that do not wait
  and unknown blocks are refused. Degrees become radians, millimetres
  metres, gripper pos a width through the vendor map q = (850 - pos)/1000
  and the L0 linkage, and the angle speed a velocity scaling of the
  description's 3.14 rad/s limit (about 0.111).
- The generator emits each distinct move as a named pose (blockly_NN, and
  zero for reset) beside poses_rad, and the step list as the plan's
  programs: block.
- A new linear_axis category and the ufactory_linear_motor type. picker
  rides its carriage in place of picker_base; the prismatic joint is
  emitted into the arm's description under its base, with its own
  JointTrajectoryController in the arm's controller manager. The hardware
  path (vendor set_linear_motor_pos) is not implemented; the type declares
  sim only.
- The cell_b layout is derived by forward kinematics from the program's
  pick and place poses: infeed_table under the pads at track 0, the belt's
  infeed under them at track 650 mm. PROVISIONAL.
- The work-piece is a 66 mm cube, the smallest whole millimetre over which
  the program's 60.9 mm close still evidences a grasp. The belt inset is
  0.055 m so that the larger part keeps its support margin in both cells.
- Validator rules: program-refused, program-pose-outside-joint-limits
  (limits copied from the vendor description into L0),
  program-pose-name-taken, program-track-*, track-backend-differs-from-its-arm,
  program-grip-never-evidences-a-grasp; the reach check is track-aware.

Tests pinned to the 50 mm part are moved to the 66 mm part, except the
re-analysis of the 2026-09-01 campaign, which keeps the 50 mm part its
trials gripped.

Co-Authored-By: Claude Opus 5.5 <noreply@anthropic.com>

File: workspace/src/cite_generated/description/cell_a_scene.urdf.xacro (robot description, xacro)
@@ -87,5 +87,5 @@
     <parent link="cite_world"/>
     <child link="beam_c1_out_base_link"/>
-    <origin xyz="1.627 0.25 0.63" rpy="0 0 0"/>
+    <origin xyz="1.63 0.25 0.63" rpy="0 0 0"/>
   </joint>
   <link name="beam_c1_out_beam"/>
@@ -121,5 +121,5 @@
     <parent link="cite_world"/>
     <child link="beam_c2_out_base_link"/>
-    <origin xyz="3.727 0.25 0.63" rpy="0 0 0"/>
+    <origin xyz="3.73 0.25 0.63" rpy="0 0 0"/>
   </joint>
   <link name="beam_c2_out_beam"/>
@@ -155,5 +155,5 @@
     <parent link="cite_world"/>
     <child link="beam_c3_out_base_link"/>
-    <origin xyz="5.75 0.25 0.63" rpy="0 0 0"/>
+    <origin xyz="5.745 0.25 0.63" rpy="0 0 0"/>
   </joint>
   <link name="beam_c3_out_beam"/>
@@ -229,5 +229,5 @@
     <parent link="conveyor_1_base_link"/>
     <child link="conveyor_1_infeed"/>
-    <origin xyz="-0.55 0 0.6" rpy="0 0 0"/>
+    <origin xyz="-0.545 0 0.6" rpy="0 0 0"/>
   </joint>
   <link name="conveyor_1_outfeed"/>
@@ -235,5 +235,5 @@
     <parent link="conveyor_1_base_link"/>
     <child link="conveyor_1_outfeed"/>
-    <origin xyz="0.55 0 0.6" rpy="0 0 0"/>
+    <origin xyz="0.545 0 0.6" rpy="0 0 0"/>
   </joint>
   <link name="conveyor_1_surface"/>
@@ -275,5 +275,5 @@
     <parent link="conveyor_2_base_link"/>
     <child link="conveyor_2_infeed"/>
-    <origin xyz="-0.55 0 0.6" rpy="0 0 0"/>
+    <origin xyz="-0.545 0 0.6" rpy="0 0 0"/>
   </joint>
   <link name="conveyor_2_outfeed"/>
@@ -281,5 +281,5 @@
     <parent link="conveyor_2_base_link"/>
     <child link="conveyor_2_outfeed"/>
-    <origin xyz="0.55 0 0.6" rpy="0 0 0"/>
+    <origin xyz="0.545 0 0.6" rpy="0 0 0"/>
   </joint>
   <link name="conveyor_2_surface"/>
@@ -321,5 +321,5 @@
     <parent link="conveyor_3_base_link"/>
     <child link="conveyor_3_infeed"/>
-    <origin xyz="-0.55 0 0.6" rpy="0 0 0"/>
+    <origin xyz="-0.545 0 0.6" rpy="0 0 0"/>
   </joint>
   <link name="conveyor_3_outfeed"/>
@@ -327,5 +327,5 @@
     <parent link="conveyor_3_base_link"/>
     <child link="conveyor_3_outfeed"/>
-    <origin xyz="0.55 0 0.6" rpy="0 0 0"/>
+    <origin xyz="0.545 0 0.6" rpy="0 0 0"/>
   </joint>
   <link name="conveyor_3_surface"/>

File: workspace/src/cite_generated/description/cell_b_picker.urdf.xacro (robot description, xacro)
@@ -17,9 +17,52 @@
        coordinate of its own. -->
   <link name="picker_mount"/>
+  <!-- The linear track this arm rides (ADR-0067). Its rail is a body in the
+       scene; its one joint is HERE, between the mount and the carriage the arm's
+       base is bolted to, so robot_state_publisher, MoveIt's robot state and its
+       collision checks all see where the arm really is. The mount stands where
+       the carriage is at stroke zero, and the axis is stated in the mount's own
+       frame, derived from the track type's direction.
+       The carriage has mass because a massless link between two joints is
+       dropped by the URDF-to-SDF converter, and the axis with it. It has no
+       collision geometry: the plate rides 5 mm above the rail's top face and is
+       drawn, not checked. -->
+  <link name="picker_track_carriage">
+    <inertial>
+      <origin xyz="0 0 -0.0025" rpy="0 0 0"/>
+      <mass value="3"/>
+      <inertia ixx="0.00640625" ixy="0" ixz="0" iyy="0.01000625" iyz="0" izz="0.0164"/>
+    </inertial>
+    <visual>
+      <origin xyz="0 0 -0.0025" rpy="0 0 0"/>
+      <geometry><box size="0.2 0.16 0.005"/></geometry>
+    </visual>
+  </link>
+  <joint name="picker_track_joint" type="prismatic">
+    <parent link="picker_mount"/>
+    <child link="picker_track_carriage"/>
+    <origin xyz="0 0 0" rpy="0 0 0"/>
+    <axis xyz="0 1 0"/>
+    <limit lower="0" upper="0.7" velocity="1" effort="500"/>
+  </joint>
+  <!-- One hardware component for the track, beside the arm's own: the same
+       controller manager loads both, and only the plugin names which machine is
+       behind it. The track's hardware path is not implemented (ADR-0067). -->
+  <ros2_control name="picker_track_joint_system" type="system">
+    <hardware>
+      <plugin>gz_ros2_control/GazeboSimSystem</plugin>
+    </hardware>
+    <joint name="picker_track_joint">
+      <command_interface name="position"/>
+      <state_interface name="position">
+        <param name="initial_value">0.0</param>
+      </state_interface>
+      <state_interface name="velocity"/>
+    </joint>
+  </ros2_control>
   <xacro:include filename="$(find xarm_description)/urdf/xarm_device_macro.xacro"/>
   <xacro:xarm_device
       add_gripper="true"
       attach_rpy="0 0 0"
-      attach_to="picker_mount"
+      attach_to="picker_track_carriage"
       attach_xyz="0 0 0"
       collision_mesh_path="file://$(find cite_description)/meshes/collision/xarm5/convex_hull"

File: workspace/src/cite_generated/description/cell_b_scene.urdf.xacro (robot description, xacro)
@@ -52,7 +52,4 @@
     <color rgba="0.28 0.34 0.42 1"/>
   </material>
-  <material name="pedestal_steel">
-    <color rgba="0.52 0.53 0.56 1"/>
-  </material>
   <material name="sensor_housing">
     <color rgba="0.78 0.62 0.1 1"/>
@@ -87,5 +84,5 @@
     <parent link="cite_world"/>
     <child link="infeed_beam_base_link"/>
-    <origin xyz="-0.475 3.25 0.63" rpy="0 0 0"/>
+    <origin xyz="-0.5 2.674 0.63" rpy="0 0 0"/>
   </joint>
   <link name="infeed_beam_beam"/>
@@ -121,5 +118,5 @@
     <parent link="cite_world"/>
     <child link="infeed_table_base_link"/>
-    <origin xyz="-0.475 3 0" rpy="0 0 0"/>
+    <origin xyz="-0.5 2.924 0" rpy="0 0 0"/>
   </joint>
   <link name="infeed_table_surface"/>
@@ -155,5 +152,5 @@
     <parent link="cite_world"/>
     <child link="outfeed_beam_base_link"/>
-    <origin xyz="1.55 3.25 0.63" rpy="0 0 0"/>
+    <origin xyz="1.805 3.31 0.665" rpy="0 0 0"/>
   </joint>
   <link name="outfeed_beam_beam"/>
@@ -189,5 +186,5 @@
     <parent link="cite_world"/>
     <child link="outfeed_table_base_link"/>
-    <origin xyz="2 3 0" rpy="0 0 0"/>
+    <origin xyz="2.26 3.06 0" rpy="0 0 0"/>
   </joint>
   <link name="outfeed_table_surface"/>
@@ -197,37 +194,31 @@
     <origin xyz="0 0 0.6" rpy="0 0 0"/>
   </joint>
-  <!-- picker_base — pedestal_600 -->
-  <link name="picker_base_base_link">
-    <inertial>
-      <!-- The body's pose names the point it stands on, so the mass sits half a
-           height above the link origin. `com_m` is measured from the box centre
-           and the tensor beside it is centroidal; declaring both at the foot
-           states a centroidal tensor about a point up to 0.3 m from the mass. -->
-      <origin xyz="0 0 0.3" rpy="0 0 0"/>
-      <mass value="40"/>
-      <inertia ixx="1.5" ixy="0"
-               ixz="0" iyy="1.5"
-               iyz="0" izz="0.6"/>
-    </inertial>
-    <visual>
-      <origin xyz="0 0 0.3" rpy="0 0 0"/>
-      <geometry><box size="0.3 0.3 0.6"/></geometry>
-      <material name="pedestal_steel"/>
-    </visual>
-    <collision>
-      <origin xyz="0 0 0.3" rpy="0 0 0"/>
-      <geometry><box size="0.3 0.3 0.6"/></geometry>
-    </collision>
-  </link>
-  <joint name="picker_base_anchor" type="fixed">
-    <parent link="cite_world"/>
-    <child link="picker_base_base_link"/>
-    <origin xyz="0 2.7 0" rpy="0 0 0"/>
-  </joint>
-  <link name="picker_base_top"/>
-  <joint name="picker_base_top_fixed" type="fixed">
-    <parent link="picker_base_base_link"/>
-    <child link="picker_base_top"/>
-    <origin xyz="0 0 0.6" rpy="0 0 0"/>
+  <!-- picker_track — ufactory_linear_motor -->
+  <link name="picker_track_base_link">
+    <inertial>
+      <!-- The body's pose names the point it stands on, so the mass sits half a
+           height above the link origin. `com_m` is measured from the box centre
+           and the tensor beside it is centroidal; declaring both at the foot
+           states a centroidal tensor about a point up to 0.3 m from the mass. -->
+      <origin xyz="0 0 0.3525" rpy="0 0 0"/>
+      <mass value="25"/>
+      <inertia ixx="1.0607" ixy="0"
+               ixz="0" iyy="3.1188"
+               iyz="0" izz="2.1086"/>
+    </inertial>
+    <visual>
+      <origin xyz="0 0 0.3525" rpy="0 0 0"/>
+      <geometry><box size="1 0.11 0.705"/></geometry>
+      <material name="conveyor_frame"/>
+    </visual>
+    <collision>
+      <origin xyz="0 0 0.3525" rpy="0 0 0"/>
+      <geometry><box size="1 0.11 0.705"/></geometry>
+    </collision>
+  </link>
+  <joint name="picker_track_anchor" type="fixed">
+    <parent link="cite_world"/>
+    <child link="picker_track_base_link"/>
+    <origin xyz="0.05 3.3 0" rpy="0 0 0"/>
   </joint>
   <!-- transfer_belt — belt_1200x400 -->
@@ -257,5 +248,5 @@
     <parent link="cite_world"/>
     <child link="transfer_belt_base_link"/>
-    <origin xyz="1.05 3 0" rpy="0 0 0"/>
+    <origin xyz="1.31 3.06 0.035" rpy="0 0 0"/>
   </joint>
   <link name="transfer_belt_infeed"/>
@@ -263,5 +254,5 @@
     <parent link="transfer_belt_base_link"/>
     <child link="transfer_belt_infeed"/>
-    <origin xyz="-0.55 0 0.6" rpy="0 0 0"/>
+    <origin xyz="-0.545 0 0.6" rpy="0 0 0"/>
   </joint>
   <link name="transfer_belt_outfeed"/>
@@ -269,5 +260,5 @@
     <parent link="transfer_belt_base_link"/>
     <child link="transfer_belt_outfeed"/>
-    <origin xyz="0.55 0 0.6" rpy="0 0 0"/>
+    <origin xyz="0.545 0 0.6" rpy="0 0 0"/>
   </joint>
   <link name="transfer_belt_surface"/>
