Commit message: refactor(model): name cell_b's assets for their roles, not for their zone
The seven `b_`-prefixed ids become role names: `picker`, `picker_base`,
`infeed_table`, `outfeed_table`, `transfer_belt`, `infeed_beam`, `outfeed_beam`.
The project owner's decision, taken after all three variants were measured: each
validates clean at all three levels for both zones and each leaves `cell_a`
byte-identical, so cost was not a discriminator and consistency was the choice.

The argument for the prefix is replaced rather than deleted, because the hazard
it names is real and a later reader will re-derive it otherwise. Asset ids are
facility-unique (`referential.py`), and joint, link, controller and `_mount`
names are built from the asset id ALONE, so a second `arm_1` collides inside a
generated artifact with no finding. A role name carries that exactly as a
zone-prefixed one does, and does not encode the zone a second time in a spelling
nothing derives and nothing validates — one that also stuttered, since generated
artifact names are `<zone>_<asset>`.

`./scripts/validate-model` regenerated: 8 artifact filenames moved to
`cell_b_picker*`, 7 artifacts' content changed, `MODEL_HASH` moved, and NO
`cell_a_*` artifact moved at all. A bare re-run then exits 0 — byte identity and
the second-interpreter check both pass — reporting 2 zone(s), 7 type(s), 22
asset(s), 8 station(s), across 16 file(s). Host suites: 1606 passed, 1 skipped.

Station ids keep their `b_` prefix: they are not asset ids, they are not what
the seven-row table covers, and nothing in the collision above applies to them.

`docs/open-work.md`'s cross-zone-reference reproduction is updated with the
rename, because it is a command a reader runs.

Co-Authored-By: Claude Opus 5 (1M context) <noreply@anthropic.com>
Claude-Session: https://claude.ai/code/session_01KSp84SbGonh1nmx9bhFYrf

File: workspace/src/cite_generated/description/cell_b_picker.urdf.xacro (robot description, xacro)
@@ -5,5 +5,5 @@
      A hand edit here is a Critical review finding (ADR-0004) and is detected by
      ./scripts/validate-model, which diffs this tree against a fresh generator run. -->
-<robot xmlns:xacro="http://ros.org/wiki/xacro" name="b_arm_1">
+<robot xmlns:xacro="http://ros.org/wiki/xacro" name="picker">
   <!-- One description per arm, spawned as its own Gazebo model.
        gz_ros2_control attaches to a MODEL, and the controller manager it creates
@@ -16,10 +16,10 @@
        generated static transform table, so this description states no world
        coordinate of its own. -->
-  <link name="b_arm_1_mount"/>
+  <link name="picker_mount"/>
   <xacro:include filename="$(find xarm_description)/urdf/xarm_device_macro.xacro"/>
   <xacro:xarm_device
       add_gripper="true"
       attach_rpy="0 0 0"
-      attach_to="b_arm_1_mount"
+      attach_to="picker_mount"
       attach_xyz="0 0 0"
       collision_mesh_path="file://$(find cite_description)/meshes/collision/xarm5/convex_hull"
@@ -28,10 +28,10 @@
       effort_control="false"
       gripper_max_drive_rate_rad_s="1"
-      hw_ns="b_arm_1"
+      hw_ns="picker"
       limited="false"
       load_gazebo_plugin="false"
       mesh_suffix="stl"
       model1300="false"
-      prefix="b_arm_1_"
+      prefix="picker_"
       robot_type="xarm"
       ros2_control_plugin="gz_ros2_control/GazeboSimSystem"
@@ -39,5 +39,5 @@
   />
   <!-- Bolt the arm to the world.
-       `create_attach_link` is false and `b_arm_1_mount` is not the name
+       `create_attach_link` is false and `picker_mount` is not the name
        the URDF-to-SDF converter anchors on, so without this the arm's root is a
        free rigid body standing on its pedestal by contact friction alone. Joint
@@ -53,14 +53,14 @@
        spawn pose in the bring-up plan; a pose here would apply it twice. -->
   <gazebo>
-    <joint name="b_arm_1_mount_world_anchor" type="fixed">
+    <joint name="picker_mount_world_anchor" type="fixed">
       <parent>world</parent>
-      <child>b_arm_1_mount</child>
+      <child>picker_mount</child>
     </joint>
   </gazebo>
   <gazebo>
     <plugin filename="gz_ros2_control-system" name="gz_ros2_control::GazeboSimROS2ControlPlugin">
-      <parameters>$(find cite_generated)/control/cell_b_b_arm_1_controllers.yaml</parameters>
+      <parameters>$(find cite_generated)/control/cell_b_picker_controllers.yaml</parameters>
       <ros>
-        <namespace>/cite/cell_b/b_arm_1</namespace>
+        <namespace>/cite/cell_b/picker</namespace>
       </ros>
     </plugin>

File: workspace/src/cite_generated/description/cell_b_scene.urdf.xacro (robot description, xacro)
@@ -24,6 +24,6 @@
        below is expressed relative to it. -->
   <link name="cite_world"/>
-  <!-- b_beam_out — break_beam -->
-  <link name="b_beam_out_base_link">
+  <!-- infeed_beam — break_beam -->
+  <link name="infeed_beam_base_link">
     <inertial>
       <!-- The body's pose names the point it stands on, so the mass sits half a
@@ -46,17 +46,50 @@
     </collision>
   </link>
-  <joint name="b_beam_out_anchor" type="fixed">
-    <parent link="cite_world"/>
-    <child link="b_beam_out_base_link"/>
-    <origin xyz="1.55 3.25 0.63" rpy="0 0 0"/>
-  </joint>
-  <link name="b_beam_out_beam"/>
-  <joint name="b_beam_out_beam_fixed" type="fixed">
-    <parent link="b_beam_out_base_link"/>
-    <child link="b_beam_out_beam"/>
+  <joint name="infeed_beam_anchor" type="fixed">
+    <parent link="cite_world"/>
+    <child link="infeed_beam_base_link"/>
+    <origin xyz="-0.475 3.25 0.63" rpy="0 0 0"/>
+  </joint>
+  <link name="infeed_beam_beam"/>
+  <joint name="infeed_beam_beam_fixed" type="fixed">
+    <parent link="infeed_beam_base_link"/>
+    <child link="infeed_beam_beam"/>
     <origin xyz="0 0 0" rpy="0 0 0"/>
   </joint>
-  <!-- b_beam_pick — break_beam -->
-  <link name="b_beam_pick_base_link">
+  <!-- infeed_table — work_table_600 -->
+  <link name="infeed_table_base_link">
+    <inertial>
+      <!-- The body's pose names the point it stands on, so the mass sits half a
+           height above the link origin. `com_m` is measured from the box centre
+           and the tensor beside it is centroidal; declaring both at the foot
+           states a centroidal tensor about a point up to 0.3 m from the mass. -->
+      <origin xyz="0 0 0.3" rpy="0 0 0"/>
+      <mass value="30"/>
+      <inertia ixx="1.8" ixy="0"
+               ixz="0" iyy="1.8"
+               iyz="0" izz="1.8"/>
+    </inertial>
+    <visual>
+      <origin xyz="0 0 0.3" rpy="0 0 0"/>
+      <geometry><box size="0.6 0.6 0.6"/></geometry>
+    </visual>
+    <collision>
+      <origin xyz="0 0 0.3" rpy="0 0 0"/>
+      <geometry><box size="0.6 0.6 0.6"/></geometry>
+    </collision>
+  </link>
+  <joint name="infeed_table_anchor" type="fixed">
+    <parent link="cite_world"/>
+    <child link="infeed_table_base_link"/>
+    <origin xyz="-0.475 3 0" rpy="0 0 0"/>
+  </joint>
+  <link name="infeed_table_surface"/>
+  <joint name="infeed_table_surface_fixed" type="fixed">
+    <parent link="infeed_table_base_link"/>
+    <child link="infeed_table_surface"/>
+    <origin xyz="0 0 0.6" rpy="0 0 0"/>
+  </joint>
+  <!-- outfeed_beam — break_beam -->
+  <link name="outfeed_beam_base_link">
     <inertial>
       <!-- The body's pose names the point it stands on, so the mass sits half a
@@ -79,17 +112,83 @@
     </collision>
   </link>
-  <joint name="b_beam_pick_anchor" type="fixed">
-    <parent link="cite_world"/>
-    <child link="b_beam_pick_base_link"/>
-    <origin xyz="-0.475 3.25 0.63" rpy="0 0 0"/>
-  </joint>
-  <link name="b_beam_pick_beam"/>
-  <joint name="b_beam_pick_beam_fixed" type="fixed">
-    <parent link="b_beam_pick_base_link"/>
-    <child link="b_beam_pick_beam"/>
+  <joint name="outfeed_beam_anchor" type="fixed">
+    <parent link="cite_world"/>
+    <child link="outfeed_beam_base_link"/>
+    <origin xyz="1.55 3.25 0.63" rpy="0 0 0"/>
+  </joint>
+  <link name="outfeed_beam_beam"/>
+  <joint name="outfeed_beam_beam_fixed" type="fixed">
+    <parent link="outfeed_beam_base_link"/>
+    <child link="outfeed_beam_beam"/>
     <origin xyz="0 0 0" rpy="0 0 0"/>
   </joint>
-  <!-- b_conveyor_1 — belt_1200x400 -->
-  <link name="b_conveyor_1_base_link">
+  <!-- outfeed_table — work_table_600 -->
+  <link name="outfeed_table_base_link">
+    <inertial>
+      <!-- The body's pose names the point it stands on, so the mass sits half a
+           height above the link origin. `com_m` is measured from the box centre
+           and the tensor beside it is centroidal; declaring both at the foot
+           states a centroidal tensor about a point up to 0.3 m from the mass. -->
+      <origin xyz="0 0 0.3" rpy="0 0 0"/>
+      <mass value="30"/>
+      <inertia ixx="1.8" ixy="0"
+               ixz="0" iyy="1.8"
+               iyz="0" izz="1.8"/>
+    </inertial>
+    <visual>
+      <origin xyz="0 0 0.3" rpy="0 0 0"/>
+      <geometry><box size="0.6 0.6 0.6"/></geometry>
+    </visual>
+    <collision>
+      <origin xyz="0 0 0.3" rpy="0 0 0"/>
+      <geometry><box size="0.6 0.6 0.6"/></geometry>
+    </collision>
+  </link>
+  <joint name="outfeed_table_anchor" type="fixed">
+    <parent link="cite_world"/>
+    <child link="outfeed_table_base_link"/>
+    <origin xyz="2 3 0" rpy="0 0 0"/>
+  </joint>
+  <link name="outfeed_table_surface"/>
+  <joint name="outfeed_table_surface_fixed" type="fixed">
+    <parent link="outfeed_table_base_link"/>
+    <child link="outfeed_table_surface"/>
+    <origin xyz="0 0 0.6" rpy="0 0 0"/>
+  </joint>
+  <!-- picker_base — pedestal_600 -->
+  <link name="picker_base_base_link">
+    <inertial>
+      <!-- The body's pose names the point it stands on, so the mass sits half a
+           height above the link origin. `com_m` is measured from the box centre
+           and the tensor beside it is centroidal; declaring both at the foot
+           states a centroidal tensor about a point up to 0.3 m from the mass. -->
+      <origin xyz="0 0 0.3" rpy="0 0 0"/>
+      <mass value="40"/>
+      <inertia ixx="1.5" ixy="0"
+               ixz="0" iyy="1.5"
+               iyz="0" izz="0.6"/>
+    </inertial>
+    <visual>
+      <origin xyz="0 0 0.3" rpy="0 0 0"/>
+      <geometry><box size="0.3 0.3 0.6"/></geometry>
+    </visual>
+    <collision>
+      <origin xyz="0 0 0.3" rpy="0 0 0"/>
+      <geometry><box size="0.3 0.3 0.6"/></geometry>
+    </collision>
+  </link>
+  <joint name="picker_base_anchor" type="fixed">
+    <parent link="cite_world"/>
+    <child link="picker_base_base_link"/>
+    <origin xyz="0 2.7 0" rpy="0 0 0"/>
+  </joint>
+  <link name="picker_base_top"/>
+  <joint name="picker_base_top_fixed" type="fixed">
+    <parent link="picker_base_base_link"/>
+    <child link="picker_base_top"/>
+    <origin xyz="0 0 0.6" rpy="0 0 0"/>
+  </joint>
+  <!-- transfer_belt — belt_1200x400 -->
+  <link name="transfer_belt_base_link">
     <inertial>
       <!-- The body's pose names the point it stands on, so the mass sits half a
@@ -112,124 +211,25 @@
     </collision>
   </link>
-  <joint name="b_conveyor_1_anchor" type="fixed">
-    <parent link="cite_world"/>
-    <child link="b_conveyor_1_base_link"/>
+  <joint name="transfer_belt_anchor" type="fixed">
+    <parent link="cite_world"/>
+    <child link="transfer_belt_base_link"/>
     <origin xyz="1.05 3 0" rpy="0 0 0"/>
   </joint>
-  <link name="b_conveyor_1_infeed"/>
-  <joint name="b_conveyor_1_infeed_fixed" type="fixed">
-    <parent link="b_conveyor_1_base_link"/>
-    <child link="b_conveyor_1_infeed"/>
+  <link name="transfer_belt_infeed"/>
+  <joint name="transfer_belt_infeed_fixed" type="fixed">
+    <parent link="transfer_belt_base_link"/>
+    <child link="transfer_belt_infeed"/>
     <origin xyz="-0.55 0 0.6" rpy="0 0 0"/>
   </joint>
-  <link name="b_conveyor_1_outfeed"/>
-  <joint name="b_conveyor_1_outfeed_fixed" type="fixed">
-    <parent link="b_conveyor_1_base_link"/>
-    <child link="b_conveyor_1_outfeed"/>
+  <link name="transfer_belt_outfeed"/>
+  <joint name="transfer_belt_outfeed_fixed" type="fixed">
+    <parent link="transfer_belt_base_link"/>
+    <child link="transfer_belt_outfeed"/>
     <origin xyz="0.55 0 0.6" rpy="0 0 0"/>
   </joint>
-  <link name="b_conveyor_1_surface"/>
-  <joint name="b_conveyor_1_surface_fixed" type="fixed">
-    <parent link="b_conveyor_1_base_link"/>
-    <child link="b_conveyor_1_surface"/>
-    <origin xyz="0 0 0.6" rpy="0 0 0"/>
-  </joint>
-  <!-- b_pedestal_1 — pedestal_600 -->
-  <link name="b_pedestal_1_base_link">
-    <inertial>
-      <!-- The body's pose names the point it stands on, so the mass sits half a
-           height above the link origin. `com_m` is measured from the box centre
-           and the tensor beside it is centroidal; declaring both at the foot
-           states a centroidal tensor about a point up to 0.3 m from the mass. -->
-      <origin xyz="0 0 0.3" rpy="0 0 0"/>
-      <mass value="40"/>
-      <inertia ixx="1.5" ixy="0"
-               ixz="0" iyy="1.5"
-               iyz="0" izz="0.6"/>
-    </inertial>
-    <visual>
-      <origin xyz="0 0 0.3" rpy="0 0 0"/>
-      <geometry><box size="0.3 0.3 0.6"/></geometry>
-    </visual>
-    <collision>
-      <origin xyz="0 0 0.3" rpy="0 0 0"/>
-      <geometry><box size="0.3 0.3 0.6"/></geometry>
-    </collision>
-  </link>
-  <joint name="b_pedestal_1_anchor" type="fixed">
-    <parent link="cite_world"/>
-    <child link="b_pedestal_1_base_link"/>
-    <origin xyz="0 2.7 0" rpy="0 0 0"/>
-  </joint>
-  <link name="b_pedestal_1_top"/>
-  <joint name="b_pedestal_1_top_fixed" type="fixed">
-    <parent link="b_pedestal_1_base_link"/>
-    <child link="b_pedestal_1_top"/>
-    <origin xyz="0 0 0.6" rpy="0 0 0"/>
-  </joint>
-  <!-- b_table_out — work_table_600 -->
-  <link name="b_table_out_base_link">
-    <inertial>
-      <!-- The body's pose names the point it stands on, so the mass sits half a
-           height above the link origin. `com_m` is measured from the box centre
-           and the tensor beside it is centroidal; declaring both at the foot
-           states a centroidal tensor about a point up to 0.3 m from the mass. -->
-      <origin xyz="0 0 0.3" rpy="0 0 0"/>
-      <mass value="30"/>
-      <inertia ixx="1.8" ixy="0"
-               ixz="0" iyy="1.8"
-               iyz="0" izz="1.8"/>
-    </inertial>
-    <visual>
-      <origin xyz="0 0 0.3" rpy="0 0 0"/>
-      <geometry><box size="0.6 0.6 0.6"/></geometry>
-    </visual>
-    <collision>
-      <origin xyz="0 0 0.3" rpy="0 0 0"/>
-      <geometry><box size="0.6 0.6 0.6"/></geometry>
-    </collision>
-  </link>
-  <joint name="b_table_out_anchor" type="fixed">
-    <parent link="cite_world"/>
-    <child link="b_table_out_base_link"/>
-    <origin xyz="2 3 0" rpy="0 0 0"/>
-  </joint>
-  <link name="b_table_out_surface"/>
-  <joint name="b_table_out_surface_fixed" type="fixed">
-    <parent link="b_table_out_base_link"/>
-    <child link="b_table_out_surface"/>
-    <origin xyz="0 0 0.6" rpy="0 0 0"/>
-  </joint>
-  <!-- b_table_pick — work_table_600 -->
-  <link name="b_table_pick_base_link">
-    <inertial>
-      <!-- The body's pose names the point it stands on, so the mass sits half a
-           height above the link origin. `com_m` is measured from the box centre
-           and the tensor beside it is centroidal; declaring both at the foot
-           states a centroidal tensor about a point up to 0.3 m from the mass. -->
-      <origin xyz="0 0 0.3" rpy="0 0 0"/>
-      <mass value="30"/>
-      <inertia ixx="1.8" ixy="0"
-               ixz="0" iyy="1.8"
-               iyz="0" izz="1.8"/>
-    </inertial>
-    <visual>
-      <origin xyz="0 0 0.3" rpy="0 0 0"/>
-      <geometry><box size="0.6 0.6 0.6"/></geometry>
-    </visual>
-    <collision>
-      <origin xyz="0 0 0.3" rpy="0 0 0"/>
-      <geometry><box size="0.6 0.6 0.6"/></geometry>
-    </collision>
-  </link>
-  <joint name="b_table_pick_anchor" type="fixed">
-    <parent link="cite_world"/>
-    <child link="b_table_pick_base_link"/>
-    <origin xyz="-0.475 3 0" rpy="0 0 0"/>
-  </joint>
-  <link name="b_table_pick_surface"/>
-  <joint name="b_table_pick_surface_fixed" type="fixed">
-    <parent link="b_table_pick_base_link"/>
-    <child link="b_table_pick_surface"/>
+  <link name="transfer_belt_surface"/>
+  <joint name="transfer_belt_surface_fixed" type="fixed">
+    <parent link="transfer_belt_base_link"/>
+    <child link="transfer_belt_surface"/>
     <origin xyz="0 0 0.6" rpy="0 0 0"/>
   </joint>

File: workspace/src/cite_generated/moveit/cell_b_picker.srdf.xacro (robot description, xacro)
@@ -5,5 +5,5 @@
      A hand edit here is a Critical review finding (ADR-0004) and is detected by
      ./scripts/validate-model, which diffs this tree against a fresh generator run. -->
-<robot xmlns:xacro="http://ros.org/wiki/xacro" name="b_arm_1">
+<robot xmlns:xacro="http://ros.org/wiki/xacro" name="picker">
   <!-- The vendor SRDF macro, invoked with our prefix — never copied. It carries
        the self-collision matrix, which the vendor computed against the vendor's
@@ -23,5 +23,5 @@
       add_gripper="true"
       dof="5"
-      prefix="b_arm_1_"
+      prefix="picker_"
       robot_type="xarm"
   />

Commit message: docs(adr): ADR-0067, the real program drives the twin and the arm rides a track
Also gives the arm's mount link mass when a track's prismatic joint hangs
under it: the URDF-to-SDF converter drops a massless link with a moving
child, and the world anchor that names it with it.

Co-Authored-By: Claude Opus 5.5 <noreply@anthropic.com>

File: workspace/src/cite_generated/description/cell_b_picker.urdf.xacro (robot description, xacro)
@@ -16,5 +16,14 @@
        generated static transform table, so this description states no world
        coordinate of its own. -->
-  <link name="picker_mount"/>
+  <!-- With mass here, and only on an arm that rides a track: the joint under
+       this link is not fixed, and the URDF-to-SDF converter drops a massless
+       link that has a moving child, together with the world anchor below that
+       names it. It is welded to the world, so the value moves nothing. -->
+  <link name="picker_mount">
+    <inertial>
+      <mass value="1"/>
+      <inertia ixx="0.001" ixy="0" ixz="0" iyy="0.001" iyz="0" izz="0.001"/>
+    </inertial>
+  </link>
   <!-- The linear track this arm rides (ADR-0067). Its rail is a body in the
        scene; its one joint is HERE, between the mount and the carriage the arm's

Commit message: fix(real-program): check a tracked arm at stroke zero, move the BT scenarios to cell_a
Review remediation for ADR-0067, on the project owner's decisions of 2026-09-29.

- R-01: `unreachable-station` checks an arm on a track with its carriage at
  stroke zero; nothing in L3/L4 moves the track. cell_b's belt infeed is then
  1.094 m from the arm (reach 0.700 m), so `b_transfer_1` declares no
  `place_to` and L4 refuses the cell_b line at plan time. Regression test
  restores the place point and expects the error.
- T-01 / owner: default grasp width is the real program's close, 60.915 mm
  (pos 550 -> 0.300 rad -> linkage), stated once with its derivation and tied
  to the program by a host test. PickAt no longer restates 45 mm; it sends 0,
  which the skill server resolves to the L0 default from the plan.
- Owner: pick_and_place, continuous_line and bringup default to cell_a;
  program_cycle defaults to cell_b and is a blocking CI step.
- R-03: the vendor joint-limit guard parses and evaluates all ten defaults.
- T-02: the track carriage has a collision box equal to its visual box; the
  generated SRDF disables the carriage/base pair.
- R-04: ADR-0067 records that a mode change mid-slide lets the counterpart
  finish its slide.

Co-Authored-By: Claude Opus 5.5 <noreply@anthropic.com>

File: workspace/src/cite_generated/description/cell_b_picker.urdf.xacro (robot description, xacro)
@@ -33,7 +33,9 @@
        frame, derived from the track type's direction.
        The carriage has mass because a massless link between two joints is
-       dropped by the URDF-to-SDF converter, and the axis with it. It has no
-       collision geometry: the plate rides 5 mm above the rail's top face and is
-       drawn, not checked. -->
+       dropped by the URDF-to-SDF converter, and the axis with it. Its collision
+       box is its visual box: the plate rides 5 mm above the rail's top face, so
+       it touches nothing at rest, and it is what an arm link swinging down past
+       the carriage is checked against. The arm's own base is bolted to its top
+       face, and the generated SRDF disables that one adjacent pair. -->
   <link name="picker_track_carriage">
     <inertial>
@@ -46,4 +48,8 @@
       <geometry><box size="0.2 0.16 0.005"/></geometry>
     </visual>
+    <collision>
+      <origin xyz="0 0 -0.0025" rpy="0 0 0"/>
+      <geometry><box size="0.2 0.16 0.005"/></geometry>
+    </collision>
   </link>
   <joint name="picker_track_joint" type="prismatic">

File: workspace/src/cite_generated/moveit/cell_b_picker.srdf.xacro (robot description, xacro)
@@ -26,3 +26,7 @@
       robot_type="xarm"
   />
+  <!-- picker_track_carriage is bolted to picker_link_base: the track's carriage carries the
+       arm's base on its top face (ADR-0067), so the two are always in contact and
+       the vendor matrix, which has never heard of a carriage, cannot say so. -->
+  <disable_collisions link1="picker_track_carriage" link2="picker_link_base" reason="Adjacent"/>
 </robot>
