Commit message: feat(model): the transfer belt wears a generated industrial visual mesh (ADR-0079)
belt_1200x400's visual is now a parametric GLB generated from its own
collision box by python -m cite_tools.visuals.conveyor: aluminium side
frames, a rubber belt over two drums with its top on the 0.600 m surface,
40x40 legs with braces and levelling feet, a geared motor under the outfeed
end and a yellow control box with a red stop cap. PBR finishes come from the
mesh, so the body names no material. Collision, inertia, frames and the
conveyor plugin are unchanged.

- ADR-0079 (Proposed) and its index row.
- The generated package derives a dependency from a body mesh URI.
- Tests: committed GLB equals a fresh generation, lies inside the box, belt
  top on the surface frame, scene draws a mesh and collides against a box;
  cite_description checks the declared body mesh is installable.
- Regenerated cite_generated.

Co-Authored-By: Claude Opus 5.5 <noreply@anthropic.com>

File: workspace/src/cite_generated/description/cell_b_scene.urdf.xacro (robot description, xacro)
@@ -237,6 +237,5 @@
     <visual>
       <origin xyz="0 0 0.3" rpy="0 0 0"/>
-      <geometry><box size="1.2 0.4 0.6"/></geometry>
-      <material name="conveyor_frame"/>
+      <geometry><mesh filename="file://$(find cite_description)/meshes/visual/conveyors/belt_1200x400.glb" scale="1 1 1"/></geometry>
     </visual>
     <collision>

Commit message: feat(model): the work tables wear a generated light-wood visual mesh (ADR-0079)
work_table_600's visual is now a GLB drawn inside its collision box: a
chamfered top whose face is the surface frame, four square legs, an apron
on all sides, and stretchers carrying a lower shelf, in two light-wood
finishes (metallic 0). The body names no material; collision, inertia and
frames are unchanged.

The generator is generalised rather than copied: cite_tools.visuals.parts
holds the shared shapes and export, conveyor and table are drawers, and
`python -m cite_tools.visuals [--write]` checks or regenerates every body
mesh, the drawer selected by the URI's directory under meshes/visual/. The
conveyor's GLB is byte-identical across the refactor.

Tests are parametrised over every body mesh (test_visual_meshes.py). The
material clip tests now use conveyor_frame, which a body still wears.
ADR-0079 (Proposed) and its index row describe both bodies and the command.

Co-Authored-By: Claude Opus 5.5 <noreply@anthropic.com>

File: workspace/src/cite_generated/description/cell_b_scene.urdf.xacro (robot description, xacro)
@@ -55,7 +55,4 @@
     <color rgba="0.78 0.62 0.1 1"/>
   </material>
-  <material name="table_top">
-    <color rgba="0.58 0.38 0.2 1"/>
-  </material>
   <!-- infeed_beam — break_beam -->
   <link name="infeed_beam_base_link">
@@ -107,6 +104,5 @@
     <visual>
       <origin xyz="0 0 0.3" rpy="0 0 0"/>
-      <geometry><box size="0.6 0.6 0.6"/></geometry>
-      <material name="table_top"/>
+      <geometry><mesh filename="file://$(find cite_description)/meshes/visual/tables/work_table_600.glb" scale="1 1 1"/></geometry>
     </visual>
     <collision>
@@ -175,6 +171,5 @@
     <visual>
       <origin xyz="0 0 0.3" rpy="0 0 0"/>
-      <geometry><box size="0.6 0.6 0.6"/></geometry>
-      <material name="table_top"/>
+      <geometry><mesh filename="file://$(find cite_description)/meshes/visual/tables/work_table_600.glb" scale="1 1 1"/></geometry>
     </visual>
     <collision>

Commit message: feat(model): the track stands on a long pick table, and both wear generated meshes (ADR-0079)
The owner's fact about the lab: the linear track and the robot stand on the
table the part is picked from, which runs from its far corner to just past
the track's end. The model drew a 0.705 m box on the floor beside a 0.6 m
table.

- infeed_table is a new work_table_1450x800 (x -0.800..0.650,
  y 2.624..3.424, 60 mm clear of the belt). Its off-centre `surface` frame
  keeps the pick point at (-0.500, 2.924, 0.600).
- picker_track's body is the rail alone (1.000 x 0.110 x 0.105), placed on
  infeed_table/surface so its foot is at (0.050, 3.300, 0.600). Its carriage
  frame is now 0.110 above the foot, so the carriage stays at 0.710 m.
- Generated arm descriptions, static frames, world and bring-up plan are
  byte-identical. Only the two bodies change, in the scene and the planning
  scene.
- Visual meshes: a `tracks/` drawer draws the rail (profile, guides, dust
  strip, end caps, motor housing, cable gland). The table drawer places
  legs from the box size, adding a middle pair past a 1.2 m bay.
- Tests extended to the new meshes. Material clip tests now use
  sensor_housing. Generate tests that assumed a 0.6 m infeed_table now use
  outfeed_table.
- ADR-0079 addendum.

Co-Authored-By: Claude Opus 5.5 <noreply@anthropic.com>

File: workspace/src/cite_generated/description/cell_b_scene.urdf.xacro (robot description, xacro)
@@ -49,7 +49,4 @@
        component a scene body wears at or under 0.8, where the multiply cannot
        clip; the reason is stated on the library itself. -->
-  <material name="conveyor_frame">
-    <color rgba="0.28 0.34 0.42 1"/>
-  </material>
   <material name="sensor_housing">
     <color rgba="0.78 0.62 0.1 1"/>
@@ -89,5 +86,5 @@
     <origin xyz="0 0 0" rpy="0 0 0"/>
   </joint>
-  <!-- infeed_table — work_table_600 -->
+  <!-- infeed_table — work_table_1450x800 -->
   <link name="infeed_table_base_link">
     <inertial>
@@ -97,16 +94,16 @@
            states a centroidal tensor about a point up to 0.3 m from the mass. -->
       <origin xyz="0 0 0.3" rpy="0 0 0"/>
-      <mass value="30"/>
-      <inertia ixx="1.8" ixy="0"
-               ixz="0" iyy="1.8"
-               iyz="0" izz="1.8"/>
-    </inertial>
-    <visual>
-      <origin xyz="0 0 0.3" rpy="0 0 0"/>
-      <geometry><mesh filename="file://$(find cite_description)/meshes/visual/tables/work_table_600.glb" scale="1 1 1"/></geometry>
-    </visual>
-    <collision>
-      <origin xyz="0 0 0.3" rpy="0 0 0"/>
-      <geometry><box size="0.6 0.6 0.6"/></geometry>
+      <mass value="80"/>
+      <inertia ixx="6.6667" ixy="0"
+               ixz="0" iyy="16.4167"
+               iyz="0" izz="18.2833"/>
+    </inertial>
+    <visual>
+      <origin xyz="0 0 0.3" rpy="0 0 0"/>
+      <geometry><mesh filename="file://$(find cite_description)/meshes/visual/tables/work_table_1450x800.glb" scale="1 1 1"/></geometry>
+    </visual>
+    <collision>
+      <origin xyz="0 0 0.3" rpy="0 0 0"/>
+      <geometry><box size="1.45 0.8 0.6"/></geometry>
     </collision>
   </link>
@@ -114,5 +111,5 @@
     <parent link="cite_world"/>
     <child link="infeed_table_base_link"/>
-    <origin xyz="-0.5 2.924 0" rpy="0 0 0"/>
+    <origin xyz="-0.075 3.024 0" rpy="0 0 0"/>
   </joint>
   <link name="infeed_table_surface"/>
@@ -120,5 +117,5 @@
     <parent link="infeed_table_base_link"/>
     <child link="infeed_table_surface"/>
-    <origin xyz="0 0 0.6" rpy="0 0 0"/>
+    <origin xyz="-0.425 -0.1 0.6" rpy="0 0 0"/>
   </joint>
   <!-- outfeed_beam — break_beam -->
@@ -196,18 +193,17 @@
            and the tensor beside it is centroidal; declaring both at the foot
            states a centroidal tensor about a point up to 0.3 m from the mass. -->
-      <origin xyz="0 0 0.3525" rpy="0 0 0"/>
-      <mass value="25"/>
-      <inertia ixx="1.0607" ixy="0"
-               ixz="0" iyy="3.1188"
-               iyz="0" izz="2.1086"/>
-    </inertial>
-    <visual>
-      <origin xyz="0 0 0.3525" rpy="0 0 0"/>
-      <geometry><box size="1 0.11 0.705"/></geometry>
-      <material name="conveyor_frame"/>
-    </visual>
-    <collision>
-      <origin xyz="0 0 0.3525" rpy="0 0 0"/>
-      <geometry><box size="1 0.11 0.705"/></geometry>
+      <origin xyz="0 0 0.0525" rpy="0 0 0"/>
+      <mass value="12"/>
+      <inertia ixx="0.023125" ixy="0"
+               ixz="0" iyy="1.011025"
+               iyz="0" izz="1.0121"/>
+    </inertial>
+    <visual>
+      <origin xyz="0 0 0.0525" rpy="0 0 0"/>
+      <geometry><mesh filename="file://$(find cite_description)/meshes/visual/tracks/ufactory_linear_motor.glb" scale="1 1 1"/></geometry>
+    </visual>
+    <collision>
+      <origin xyz="0 0 0.0525" rpy="0 0 0"/>
+      <geometry><box size="1 0.11 0.105"/></geometry>
     </collision>
   </link>
@@ -215,5 +211,5 @@
     <parent link="cite_world"/>
     <child link="picker_track_base_link"/>
-    <origin xyz="0.05 3.3 0" rpy="0 0 0"/>
+    <origin xyz="0.05 3.3 0.6" rpy="0 0 0"/>
   </joint>
   <!-- transfer_belt — belt_1200x400 -->

Commit message: feat(model): the outfeed table stands closer to the belt and lower (ADR-0079)
At the owner's request: outfeed_table moves in from a 50 mm to a 25 mm gap
from the belt's end (centre x 2.260 -> 2.235). It was asked for at about
15 mm, but 20 mm is the minimum `insufficient-clearance` accepts, and exactly
20 mm still warns in floating point. work_table_600, now used only by
outfeed_table, is 0.570 m tall: box, `surface` frame and inertia follow, and
its generated mesh follows the box. Its surface is 65 mm under the belt's.
Two generate tests that pinned the old values are updated.

Co-Authored-By: Claude Opus 5.5 <noreply@anthropic.com>

File: workspace/src/cite_generated/description/cell_b_scene.urdf.xacro (robot description, xacro)
@@ -160,17 +160,17 @@
            and the tensor beside it is centroidal; declaring both at the foot
            states a centroidal tensor about a point up to 0.3 m from the mass. -->
-      <origin xyz="0 0 0.3" rpy="0 0 0"/>
+      <origin xyz="0 0 0.285" rpy="0 0 0"/>
       <mass value="30"/>
-      <inertia ixx="1.8" ixy="0"
-               ixz="0" iyy="1.8"
+      <inertia ixx="1.71225" ixy="0"
+               ixz="0" iyy="1.71225"
                iyz="0" izz="1.8"/>
     </inertial>
     <visual>
-      <origin xyz="0 0 0.3" rpy="0 0 0"/>
+      <origin xyz="0 0 0.285" rpy="0 0 0"/>
       <geometry><mesh filename="file://$(find cite_description)/meshes/visual/tables/work_table_600.glb" scale="1 1 1"/></geometry>
     </visual>
     <collision>
-      <origin xyz="0 0 0.3" rpy="0 0 0"/>
-      <geometry><box size="0.6 0.6 0.6"/></geometry>
+      <origin xyz="0 0 0.285" rpy="0 0 0"/>
+      <geometry><box size="0.6 0.6 0.57"/></geometry>
     </collision>
   </link>
@@ -178,5 +178,5 @@
     <parent link="cite_world"/>
     <child link="outfeed_table_base_link"/>
-    <origin xyz="2.26 3.06 0" rpy="0 0 0"/>
+    <origin xyz="2.235 3.06 0" rpy="0 0 0"/>
   </joint>
   <link name="outfeed_table_surface"/>
@@ -184,5 +184,5 @@
     <parent link="outfeed_table_base_link"/>
     <child link="outfeed_table_surface"/>
-    <origin xyz="0 0 0.6" rpy="0 0 0"/>
+    <origin xyz="0 0 0.57" rpy="0 0 0"/>
   </joint>
   <!-- picker_track — ufactory_linear_motor -->

Commit message: feat(model): the outfeed table is 0.550 m tall (ADR-0079)
At the owner's request, a little lower again: work_table_600's box, surface
frame and inertia follow, and its generated mesh follows the box. Its surface
is now 85 mm under the belt's.

Co-Authored-By: Claude Opus 5.5 <noreply@anthropic.com>

File: workspace/src/cite_generated/description/cell_b_scene.urdf.xacro (robot description, xacro)
@@ -160,17 +160,17 @@
            and the tensor beside it is centroidal; declaring both at the foot
            states a centroidal tensor about a point up to 0.3 m from the mass. -->
-      <origin xyz="0 0 0.285" rpy="0 0 0"/>
+      <origin xyz="0 0 0.275" rpy="0 0 0"/>
       <mass value="30"/>
-      <inertia ixx="1.71225" ixy="0"
-               ixz="0" iyy="1.71225"
+      <inertia ixx="1.65625" ixy="0"
+               ixz="0" iyy="1.65625"
                iyz="0" izz="1.8"/>
     </inertial>
     <visual>
-      <origin xyz="0 0 0.285" rpy="0 0 0"/>
+      <origin xyz="0 0 0.275" rpy="0 0 0"/>
       <geometry><mesh filename="file://$(find cite_description)/meshes/visual/tables/work_table_600.glb" scale="1 1 1"/></geometry>
     </visual>
     <collision>
-      <origin xyz="0 0 0.285" rpy="0 0 0"/>
-      <geometry><box size="0.6 0.6 0.57"/></geometry>
+      <origin xyz="0 0 0.275" rpy="0 0 0"/>
+      <geometry><box size="0.6 0.6 0.55"/></geometry>
     </collision>
   </link>
@@ -184,5 +184,5 @@
     <parent link="outfeed_table_base_link"/>
     <child link="outfeed_table_surface"/>
-    <origin xyz="0 0 0.57" rpy="0 0 0"/>
+    <origin xyz="0 0 0.55" rpy="0 0 0"/>
   </joint>
   <!-- picker_track — ufactory_linear_motor -->

Commit message: feat(model): remove the unread break beams from cell_b (ADR-0079)
The owner asked for the two yellow beam housings to look better, or to go
if they do nothing. Nothing in the main tree acts on them:
- the program, cite_twin, the console and both scenarios read neither their
  topics nor the plan's sensors;
- the flow's station triggers and the bridged level topics had no reader;
- the beam-triggered line left with ADR-0069.

So infeed_beam, outfeed_beam, the break_beam type, both station triggers and
the sensor_housing material are removed. The generated world, plan, scene,
frames, flow and planning scene drop them.

Beams can still be declared: the schema, the validators, the generators, the
bridge and the cite_break_beam plugin all stay. The tests of that support
restore the cell's former beams from tools/tests/fixtures/beams/, or add a
plan entry of their own.

program_cycle found the one real dependency: tests/scenarios/_cell.py took
the part name as the belts' <carry> intersected with the beams' <watch>,
which is empty without beams. It now uses the carry list alone when no beam
watches.

Docs that showed a beam topic now show a belt topic. The glossary entry is
updated, open-work #81 and its neighbour get a one-line note, and ADR-0079
gets an addendum.

Co-Authored-By: Claude Opus 5.5 <noreply@anthropic.com>

File: workspace/src/cite_generated/description/cell_b_scene.urdf.xacro (robot description, xacro)
@@ -24,66 +24,4 @@
        below is expressed relative to it. -->
   <link name="cite_world"/>
-  <!-- The appearances the bodies below wear, defined once each and referenced by
-       name. Every value is resolved from the facility's material library in L0;
-       nothing here is authored.
-       WHY THESE EXIST AT ALL. Until 2026-09-28 every visual in this file was a
-       bare <geometry> and the cell rendered black, while L0 had carried a
-       material name on each of those bodies the whole time and nothing resolved
-       it.
-       DEFINED HERE AND REFERENCED BELOW, rather than repeated inside each
-       <visual>. urdfdom resolves a name-only <material> against the robot-scope
-       map, so this is the form in which one colour is written once per document
-       — and repeating a definition makes urdfdom warn that the material is not
-       unique and keep whichever it saw first.
-       ONE COLOUR, WHERE L0 DECLARES TWO, AND THE DIFFUSE IS THE ONE THAT SURVIVES.
-       URDF has a single <color> per material and no ambient term. Measured in
-       this project's container on 2026-09-28 with `gz sdf -p` over a probe URDF:
-       sdformat copies this rgba onto BOTH the SDF ambient and the SDF diffuse,
-       after multiplying the three colour components by 1.25 and clamping each at
-       1.0, with alpha untouched. So the declared ambient reaches nothing on this
-       path and the declared diffuse is shown 25% brighter.
-       That is recorded and NOT compensated for. Dividing by 1.25 here would put
-       an undeclared constant in this template that tracks an upstream
-       implementation detail, and what it would buy is cosmetic — nothing in this
-       repository measures a colour. What the library does instead is keep every
-       component a scene body wears at or under 0.8, where the multiply cannot
-       clip; the reason is stated on the library itself. -->
-  <material name="sensor_housing">
-    <color rgba="0.78 0.62 0.1 1"/>
-  </material>
-  <!-- infeed_beam — break_beam -->
-  <link name="infeed_beam_base_link">
-    <inertial>
-      <!-- The body's pose names the point it stands on, so the mass sits half a
-           height above the link origin. `com_m` is measured from the box centre
-           and the tensor beside it is centroidal; declaring both at the foot
-           states a centroidal tensor about a point up to 0.3 m from the mass. -->
-      <origin xyz="0 0 0.06" rpy="0 0 0"/>
-      <mass value="0.25"/>
-      <inertia ixx="0.00033333" ixy="0"
-               ixz="0" iyy="0.00033333"
-               iyz="0" izz="6.667e-05"/>
-    </inertial>
-    <visual>
-      <origin xyz="0 0 0.06" rpy="0 0 0"/>
-      <geometry><box size="0.04 0.04 0.12"/></geometry>
-      <material name="sensor_housing"/>
-    </visual>
-    <collision>
-      <origin xyz="0 0 0.06" rpy="0 0 0"/>
-      <geometry><box size="0.04 0.04 0.12"/></geometry>
-    </collision>
-  </link>
-  <joint name="infeed_beam_anchor" type="fixed">
-    <parent link="cite_world"/>
-    <child link="infeed_beam_base_link"/>
-    <origin xyz="-0.5 2.674 0.63" rpy="0 0 0"/>
-  </joint>
-  <link name="infeed_beam_beam"/>
-  <joint name="infeed_beam_beam_fixed" type="fixed">
-    <parent link="infeed_beam_base_link"/>
-    <child link="infeed_beam_beam"/>
-    <origin xyz="0 0 0" rpy="0 0 0"/>
-  </joint>
   <!-- infeed_table — work_table_1450x800 -->
   <link name="infeed_table_base_link">
@@ -118,38 +56,4 @@
     <child link="infeed_table_surface"/>
     <origin xyz="-0.425 -0.1 0.6" rpy="0 0 0"/>
-  </joint>
-  <!-- outfeed_beam — break_beam -->
-  <link name="outfeed_beam_base_link">
-    <inertial>
-      <!-- The body's pose names the point it stands on, so the mass sits half a
-           height above the link origin. `com_m` is measured from the box centre
-           and the tensor beside it is centroidal; declaring both at the foot
-           states a centroidal tensor about a point up to 0.3 m from the mass. -->
-      <origin xyz="0 0 0.06" rpy="0 0 0"/>
-      <mass value="0.25"/>
-      <inertia ixx="0.00033333" ixy="0"
-               ixz="0" iyy="0.00033333"
-               iyz="0" izz="6.667e-05"/>
-    </inertial>
-    <visual>
-      <origin xyz="0 0 0.06" rpy="0 0 0"/>
-      <geometry><box size="0.04 0.04 0.12"/></geometry>
-      <material name="sensor_housing"/>
-    </visual>
-    <collision>
-      <origin xyz="0 0 0.06" rpy="0 0 0"/>
-      <geometry><box size="0.04 0.04 0.12"/></geometry>
-    </collision>
-  </link>
-  <joint name="outfeed_beam_anchor" type="fixed">
-    <parent link="cite_world"/>
-    <child link="outfeed_beam_base_link"/>
-    <origin xyz="1.805 3.31 0.665" rpy="0 0 0"/>
-  </joint>
-  <link name="outfeed_beam_beam"/>
-  <joint name="outfeed_beam_beam_fixed" type="fixed">
-    <parent link="outfeed_beam_base_link"/>
-    <child link="outfeed_beam_beam"/>
-    <origin xyz="0 0 0" rpy="0 0 0"/>
   </joint>
   <!-- outfeed_table — work_table_600 -->
